Commit message: wrist

File: hand_robot_ws/src/hand_description/urdf/wrist.xacro (robot description, xacro)
@@ -30,4 +30,31 @@
       <material>Gazebo/White</material>
     </gazebo>
+    <!-- Joint entre bearing et wrist -->
+    <joint name="wrist_bearing_joint" type="fixed">
+      <parent link="bearing_link"/>
+      <child link="wrist_link"/>
+      <origin xyz="0 0 0" rpy="0 0 0"/>
+    </joint>
+    <!-- wrist link -->
+    <link name="wrist_link">
+      <visual>
+        <geometry>
+          <mesh filename="package://hand_description/meshes/wrist.stl" scale="0.001 0.001 0.001"/>
+        </geometry>
+        <material name="white"/>
+        <origin xyz="-0.005 0.072 -0.071" rpy="0 ${90 * pi / 180} 0"/>
+      </visual>
+      <collision>
+          <geometry>
+            <mesh filename="package://hand_description/meshes/wrist.stl" scale="0.001 0.001 0.001"/>
+        </geometry>
+        <origin xyz="0 0 0" rpy="0 0 0"/>
+      </collision>
+      <xacro:cylinder_inertia mass="0.1" radius="0.02" length="0.04"/>
+    </link>
+    <!-- Color Gazebo for wrist -->
+    <gazebo reference="wrist_link">
+      <material>Gazebo/White</material>
+    </gazebo>
   </xacro:macro>
 </robot>
