Commit message: palm+servo

File: hand_robot_ws/src/hand_description/urdf/palm.xacro (robot description, xacro)
@@ -78,4 +78,244 @@
       <xacro:cylinder_inertia mass="0.5" radius="0.08" length="0.25"/>
     </link>
+    <!-- Joint entre palm et servo -->
+    <joint name="palm_sg90_index_joint" type="fixed">
+      <parent link="palm_link"/>
+      <child link="sg90_index_link"/>
+      <origin xyz="0.077 0.002 0.0075" rpy="${180 * pi / 180} ${0 * pi / 180} ${-100 * pi / 180}"/>
+    </joint>
+    <!-- middle base left -->
+    <link name="sg90_index_link">
+      <visual>
+        <geometry>
+          <mesh filename="package://hand_description/meshes/SG90.stl" scale="0.001 0.001 0.001"/>
+        </geometry>
+        <material name="black"/>
+        <origin xyz="-0.0025 -0.001 0" rpy="${-3 * pi / 180} ${10 * pi / 180} ${2 * pi / 180}"/>
+      </visual>
+      <collision>
+        <geometry>
+          <mesh filename="package://hand_description/meshes/SG90.stl" scale="0.001 0.001 0.001"/>
+        </geometry>
+        <origin xyz="0 0 0" rpy="0 0 0"/>
+      </collision>
+      <xacro:cylinder_inertia mass="0.5" radius="0.08" length="0.25"/>
+    </link>
+    <!-- Joint entre palm et servo -->
+    <joint name="sg90_arm_index_joint" type="revolute">
+      <parent link="sg90_index_link"/>
+      <child link="sg90_arm_index_link"/>
+      <origin xyz="0.0028 0.006 0.03" rpy="${-3 * pi / 180} ${10 * pi / 180} ${2 * pi / 180}"/>
+      <axis xyz="0 0 1"/>
+      <limit effort="10.0" lower="${-70 * pi / 180}" upper="${50 * pi / 180}" velocity="0.3"/>
+    </joint>
+    <!-- middle base left -->
+    <link name="sg90_arm_index_link">
+      <visual>
+        <geometry>
+          <mesh filename="package://hand_description/meshes/SG90_arm.stl" scale="0.001 0.001 0.001"/>
+        </geometry>
+        <material name="orange"/>
+        <origin xyz="0.0067 0.0003 0" rpy="${180 * pi / 180} ${0 * pi / 180} ${90 * pi / 180}"/>
+      </visual>
+      <collision>
+        <geometry>
+          <mesh filename="package://hand_description/meshes/SG90_arm.stl" scale="0.001 0.001 0.001"/>
+        </geometry>
+        <origin xyz="0 0 0" rpy="0 0 0"/>
+      </collision>
+      <xacro:cylinder_inertia mass="0.5" radius="0.08" length="0.25"/>
+    </link>
+    <!-- Joint entre palm et servo -->
+    <joint name="palm_sg90_middle_joint" type="fixed">
+      <parent link="palm_link"/>
+      <child link="sg90_middle_link"/>
+      <origin xyz="0.08 0.026 0.004" rpy="${180 * pi / 180} ${5 * pi / 180} ${-95 * pi / 180}"/>
+    </joint>
+    <!-- middle base left -->
+    <link name="sg90_middle_link">
+      <visual>
+        <geometry>
+          <mesh filename="package://hand_description/meshes/SG90.stl" scale="0.001 0.001 0.001"/>
+        </geometry>
+        <material name="black"/>
+        <origin xyz="-0.0025 -0.001 0" rpy="${-3 * pi / 180} ${10 * pi / 180} ${2 * pi / 180}"/>
+      </visual>
+      <collision>
+        <geometry>
+          <mesh filename="package://hand_description/meshes/SG90.stl" scale="0.001 0.001 0.001"/>
+        </geometry>
+        <origin xyz="0 0 0" rpy="0 0 0"/>
+      </collision>
+      <xacro:cylinder_inertia mass="0.5" radius="0.08" length="0.25"/>
+    </link>
+    <!-- Joint entre palm et servo -->
+    <joint name="sg90_arm_middle_joint" type="revolute">
+      <parent link="sg90_middle_link"/>
+      <child link="sg90_arm_middle_link"/>
+      <origin xyz="0.0028 0.006 0.03" rpy="${-3 * pi / 180} ${10 * pi / 180} ${2 * pi / 180}"/>
+      <axis xyz="0 0 1"/>
+      <limit effort="10.0" lower="${-70 * pi / 180}" upper="${50 * pi / 180}" velocity="0.3"/>
+    </joint>
+    <!-- middle base left -->
+    <link name="sg90_arm_middle_link">
+      <visual>
+        <geometry>
+          <mesh filename="package://hand_description/meshes/SG90_arm.stl" scale="0.001 0.001 0.001"/>
+        </geometry>
+        <material name="orange"/>
+        <origin xyz="0.0067 0.0003 0" rpy="${180 * pi / 180} ${0 * pi / 180} ${90 * pi / 180}"/>
+      </visual>
+      <collision>
+        <geometry>
+          <mesh filename="package://hand_description/meshes/SG90_arm.stl" scale="0.001 0.001 0.001"/>
+        </geometry>
+        <origin xyz="0 0 0" rpy="0 0 0"/>
+      </collision>
+      <xacro:cylinder_inertia mass="0.5" radius="0.08" length="0.25"/>
+    </link>
+    <!-- Joint entre palm et servo -->
+    <joint name="palm_sg90_ring_joint" type="fixed">
+      <parent link="palm_link"/>
+      <child link="sg90_ring_link"/>
+      <origin xyz="0.079 0.054 0.001" rpy="${180 * pi / 180} ${10 * pi / 180} ${-87 * pi / 180}"/>
+    </joint>
+    <!-- middle base left -->
+    <link name="sg90_ring_link">
+      <visual>
+        <geometry>
+          <mesh filename="package://hand_description/meshes/SG90.stl" scale="0.001 0.001 0.001"/>
+        </geometry>
+        <material name="black"/>
+        <origin xyz="-0.0025 -0.001 0" rpy="${-3 * pi / 180} ${10 * pi / 180} ${2 * pi / 180}"/>
+      </visual>
+      <collision>
+        <geometry>
+          <mesh filename="package://hand_description/meshes/SG90.stl" scale="0.001 0.001 0.001"/>
+        </geometry>
+        <origin xyz="0 0 0" rpy="0 0 0"/>
+      </collision>
+      <xacro:cylinder_inertia mass="0.5" radius="0.08" length="0.25"/>
+    </link>
+    <!-- Joint entre palm et servo -->
+    <joint name="sg90_arm_ring_joint" type="revolute">
+      <parent link="sg90_ring_link"/>
+      <child link="sg90_arm_ring_link"/>
+      <origin xyz="0.0028 0.006 0.03" rpy="${-3 * pi / 180} ${10 * pi / 180} ${2 * pi / 180}"/>
+      <axis xyz="0 0 1"/>
+      <limit effort="10.0" lower="${-70 * pi / 180}" upper="${50 * pi / 180}" velocity="0.3"/>
+    </joint>
+    <!-- middle base left -->
+    <link name="sg90_arm_ring_link">
+      <visual>
+        <geometry>
+          <mesh filename="package://hand_description/meshes/SG90_arm.stl" scale="0.001 0.001 0.001"/>
+        </geometry>
+        <material name="orange"/>
+        <origin xyz="0.0067 0.0003 0" rpy="${180 * pi / 180} ${0 * pi / 180} ${90 * pi / 180}"/>
+      </visual>
+      <collision>
+        <geometry>
+          <mesh filename="package://hand_description/meshes/SG90_arm.stl" scale="0.001 0.001 0.001"/>
+        </geometry>
+        <origin xyz="0 0 0" rpy="0 0 0"/>
+      </collision>
+      <xacro:cylinder_inertia mass="0.5" radius="0.08" length="0.25"/>
+    </link>
+    <!-- Joint entre palm et servo -->
+    <joint name="palm_sg90_pinky_joint" type="fixed">
+      <parent link="palm_link"/>
+      <child link="sg90_pinky_link"/>
+      <origin xyz="0.046 0.045 0.004" rpy="${180 * pi / 180} ${10 * pi / 180} ${-178 * pi / 180}"/>
+    </joint>
+    <!-- middle base left -->
+    <link name="sg90_pinky_link">
+      <visual>
+        <geometry>
+          <mesh filename="package://hand_description/meshes/SG90.stl" scale="0.001 0.001 0.001"/>
+        </geometry>
+        <material name="black"/>
+        <origin xyz="-0.0025 -0.001 0" rpy="${-3 * pi / 180} ${10 * pi / 180} ${2 * pi / 180}"/>
+      </visual>
+      <collision>
+        <geometry>
+          <mesh filename="package://hand_description/meshes/SG90.stl" scale="0.001 0.001 0.001"/>
+        </geometry>
+        <origin xyz="0 0 0" rpy="0 0 0"/>
+      </collision>
+      <xacro:cylinder_inertia mass="0.5" radius="0.08" length="0.25"/>
+    </link>
+    <!-- Joint entre palm et servo -->
+    <joint name="sg90_arm_pinky_joint" type="revolute">
+      <parent link="sg90_pinky_link"/>
+      <child link="sg90_arm_pinky_link"/>
+      <origin xyz="0.0028 0.006 0.03" rpy="${-3 * pi / 180} ${10 * pi / 180} ${92 * pi / 180}"/>
+      <axis xyz="0 0 1"/>
+      <limit effort="10.0" lower="${-70 * pi / 180}" upper="${30 * pi / 180}" velocity="0.3"/>
+    </joint>
+    <!-- middle base left -->
+    <link name="sg90_arm_pinky_link">
+      <visual>
+        <geometry>
+          <mesh filename="package://hand_description/meshes/SG90_arm.stl" scale="0.001 0.001 0.001"/>
+        </geometry>
+        <material name="orange"/>
+        <origin xyz="0.0067 0.0003 0" rpy="${180 * pi / 180} ${0 * pi / 180} ${90 * pi / 180}"/>
+      </visual>
+      <collision>
+        <geometry>
+          <mesh filename="package://hand_description/meshes/SG90_arm.stl" scale="0.001 0.001 0.001"/>
+        </geometry>
+        <origin xyz="0 0 0" rpy="0 0 0"/>
+      </collision>
+      <xacro:cylinder_inertia mass="0.5" radius="0.08" length="0.25"/>
+    </link>
+    <!-- Joint entre palm et servo -->
+    <joint name="palm_sg90_thumb_joint" type="fixed">
+      <parent link="palm_link"/>
+      <child link="sg90_thumb_link"/>
+      <origin xyz="0.051 0.015 0.007" rpy="${170 * pi / 180} ${10 * pi / 180} ${2 * pi / 180}"/>
+    </joint>
+    <!-- middle base left -->
+    <link name="sg90_thumb_link">
+      <visual>
+        <geometry>
+          <mesh filename="package://hand_description/meshes/SG90.stl" scale="0.001 0.001 0.001"/>
+        </geometry>
+        <material name="black"/>
+        <origin xyz="-0.0025 -0.001 0" rpy="${-3 * pi / 180} ${10 * pi / 180} ${2 * pi / 180}"/>
+      </visual>
+      <collision>
+        <geometry>
+          <mesh filename="package://hand_description/meshes/SG90.stl" scale="0.001 0.001 0.001"/>
+        </geometry>
+        <origin xyz="0 0 0" rpy="0 0 0"/>
+      </collision>
+      <xacro:cylinder_inertia mass="0.5" radius="0.08" length="0.25"/>
+    </link>
+    <!-- Joint entre palm et servo -->
+    <joint name="sg90_arm_thumb_joint" type="revolute">
+      <parent link="sg90_thumb_link"/>
+      <child link="sg90_arm_thumb_link"/>
+      <origin xyz="0.0028 0.006 0.03" rpy="${-3 * pi / 180} ${10 * pi / 180} ${92 * pi / 180}"/>
+      <axis xyz="0 0 1"/>
+      <limit effort="10.0" lower="${0 * pi / 180}" upper="${90 * pi / 180}" velocity="0.3"/>
+    </joint>
+    <!-- middle base left -->
+    <link name="sg90_arm_thumb_link">
+      <visual>
+        <geometry>
+          <mesh filename="package://hand_description/meshes/SG90_arm.stl" scale="0.001 0.001 0.001"/>
+        </geometry>
+        <material name="orange"/>
+        <origin xyz="0.0067 0.0003 0" rpy="${180 * pi / 180} ${0 * pi / 180} ${90 * pi / 180}"/>
+      </visual>
+      <collision>
+        <geometry>
+          <mesh filename="package://hand_description/meshes/SG90_arm.stl" scale="0.001 0.001 0.001"/>
+        </geometry>
+        <origin xyz="0 0 0" rpy="0 0 0"/>
+      </collision>
+      <xacro:cylinder_inertia mass="0.5" radius="0.08" length="0.25"/>
+    </link>
   </xacro:macro>
 </robot>
