Commit message: forearm

File: hand_robot_ws/src/hand_description/urdf/hand.xacro (robot description, xacro)
@@ -3,6 +3,27 @@
   <!-- Import de tous les composants -->
   <xacro:include filename="$(find hand_description)/urdf/common.xacro"/>
-  <xacro:include filename="$(find hand_description)/urdf/index.xacro"/>
-  <!-- Instanciation de la base mobile -->
-  <xacro:index/>
+  <xacro:include filename="$(find hand_description)/urdf/ros2_control.xacro"/>
+  <xacro:include filename="$(find hand_description)/urdf/forearm.xacro"/>
+  <xacro:include filename="$(find hand_description)/urdf/wrist.xacro"/>
+  <!-- <xacro:include filename="$(find hand_description)/urdf/palm.xacro"/> -->
+  <!-- <xacro:include filename="$(find hand_description)/urdf/index.xacro"/> -->
+  <!-- <xacro:include filename="$(find hand_description)/urdf/middle.xacro"/> -->
+  <link name="base_footprint"></link>
+  <xacro:forearm parent="base_footprint">
+    <origin xyz="0 0 0" rpy="0 0 0"/>
+  </xacro:forearm>
+  <xacro:wrist parent="horn_link">
+    <origin xyz="0 0 0" rpy="0 ${90 * pi / 180} 0"/>
+  </xacro:wrist>
+  <!-- ros2_control configuration -->
+  <xacro:hand_ros2_control name="HandController" initial_positions_file=""/>
+  <!-- <xacro:palm parent="base_footprint">
+    <origin xyz="0 0 0" rpy="0 0 0"/>
+  </xacro:palm>
+  <xacro:index parent="palm_link">
+    <origin xyz="0 0.03 0.15" rpy="0 0 ${180 * pi / 180}"/>
+  </xacro:index> -->
+  <!-- <xacro:middle parent="base_footprint">
+    <origin xyz="0 0.03 0" rpy="0 0 0"/>
+  </xacro:middle> -->
 </robot>

File: hand_robot_ws/src/hand_description/urdf/index.xacro (robot description, xacro)
@@ -2,12 +2,10 @@
 <robot xmlns:xacro="http://www.ros.org/wiki/xacro">
   <!-- Index of the hand -->
-  <xacro:macro name="index">
-    <!-- Base footprint - projection au sol -->
-    <link name="base_footprint"/>
+  <xacro:macro name="index" params="parent *origin">
     <!-- Joint entre base_footprint et base_link -->
-    <joint name="base_joint" type="fixed">
-      <parent link="base_footprint"/>
+    <joint name="index_base_joint_fixed" type="fixed">
+      <parent link="${parent}"/>
       <child link="index_base_left_link"/>
-      <origin xyz="0 0 0" rpy="0 0 0"/>
+      <xacro:insert_block name="origin"/>
     </joint>
     <!-- index base left -->

Commit message: palm

File: hand_robot_ws/src/hand_description/urdf/hand.xacro (robot description, xacro)
@@ -6,5 +6,5 @@
   <xacro:include filename="$(find hand_description)/urdf/forearm.xacro"/>
   <xacro:include filename="$(find hand_description)/urdf/wrist.xacro"/>
-  <!-- <xacro:include filename="$(find hand_description)/urdf/palm.xacro"/> -->
+  <xacro:include filename="$(find hand_description)/urdf/palm.xacro"/>
   <!-- <xacro:include filename="$(find hand_description)/urdf/index.xacro"/> -->
   <!-- <xacro:include filename="$(find hand_description)/urdf/middle.xacro"/> -->
@@ -16,10 +16,10 @@
     <origin xyz="0 0 0" rpy="0 ${90 * pi / 180} 0"/>
   </xacro:wrist>
+  <xacro:palm parent="wrist_link">
+    <origin xyz="0.041 -0.035 0.001" rpy="0 0 0"/>
+  </xacro:palm>
   <!-- ros2_control configuration -->
   <xacro:hand_ros2_control name="HandController" initial_positions_file=""/>
-  <!-- <xacro:palm parent="base_footprint">
-    <origin xyz="0 0 0" rpy="0 0 0"/>
-  </xacro:palm>
-  <xacro:index parent="palm_link">
+  <!-- <xacro:index parent="palm_link">
     <origin xyz="0 0.03 0.15" rpy="0 0 ${180 * pi / 180}"/>
   </xacro:index> -->

File: hand_robot_ws/src/hand_description/urdf/palm.xacro (robot description, xacro)
@@ -3,8 +3,10 @@
   <!-- middle of the hand -->
   <xacro:macro name="palm" params="parent *origin">
-    <!-- Joint entre base_footprint et palm -->
-    <joint name="palm_base_joint_fixed" type="fixed">
+    <!-- Joint entre wrist et palm -->
+    <joint name="wrist_palm_joint" type="revolute">
       <parent link="${parent}"/>
       <child link="palm_link"/>
+      <axis xyz="0 1 0"/>
+      <limit effort="10.0" lower="${-90 * pi / 180}" upper="${90 * pi / 180}" velocity="0.3"/>
       <xacro:insert_block name="origin"/>
     </joint>
@@ -16,5 +18,5 @@
         </geometry>
         <material name="white"/>
-        <origin xyz="0 0 0" rpy="${10 * pi / 180} ${-10 * pi / 180} ${65 * pi / 180}"/>
+        <origin xyz="-0.022 0.02 0.004" rpy="${90 * pi / 180} ${-153 * pi / 180} ${95.5 * pi / 180}"/>
       </visual>
       <collision>
@@ -26,4 +28,56 @@
       <xacro:cylinder_inertia mass="0.5" radius="0.08" length="0.25"/>
     </link>
+    <!-- Joint entre palm et servo -->
+    <joint name="palm_servo_joint" type="fixed">
+      <parent link="palm_link"/>
+      <child link="servo_2_link"/>
+      <origin xyz="0.01 0.047 0.001" rpy="${90 * pi / 180} ${180 * pi / 180} ${0 * pi / 180}"/>
+    </joint>
+    <!-- Servo link -->
+    <link name="servo_2_link">
+      <visual>
+        <geometry>
+          <mesh filename="package://hand_description/meshes/Servo_Hitec_HS_645MG.stl" scale="0.001 0.001 0.001"/>
+        </geometry>
+        <material name="black"/>
+        <origin xyz="0 0 0" rpy="0 0 0"/>
+      </visual>
+      <collision>
+        <geometry>
+          <mesh filename="package://hand_description/meshes/Servo_Hitec_HS_645MG.stl" scale="0.001 0.001 0.001"/>
+        </geometry>
+        <origin xyz="0 0 0" rpy="0 0 0"/>
+      </collision>
+      <xacro:cylinder_inertia mass="0.1" radius="0.02" length="0.04"/>
+    </link>
+    <!-- Joint entre servo et horn (revolute pour rotation)-->
+    <joint name="servo_horn_2_joint" type="revolute">
+      <parent link="servo_2_link"/>
+      <child link="horn_2_link"/>
+      <origin xyz="0.01 0 0.045" rpy="${180 * pi / 180} 0 0"/>
+      <axis xyz="0 0 1"/>
+      <limit effort="10.0" lower="${-180 * pi / 180}" upper="${180 * pi / 180}" velocity="0.3"/>
+    </joint>
+    <!-- Servo link -->
+    <link name="horn_2_link">
+      <visual>
+        <geometry>
+          <mesh filename="package://hand_description/meshes/servo_circle_horn.stl" scale="0.001 0.001 0.001"/>
+        </geometry>
+        <material name="white"/>
+        <origin xyz="0 0 0" rpy="0 0 0"/>
+      </visual>
+      <collision>
+          <geometry>
+            <mesh filename="package://hand_description/meshes/servo_circle_horn.stl" scale="0.001 0.001 0.001"/>
+        </geometry>
+        <origin xyz="0 0 0" rpy="0 0 0"/>
+      </collision>
+      <xacro:cylinder_inertia mass="0.1" radius="0.02" length="0.04"/>
+    </link>
+    <!-- Color Gazebo for servo -->
+    <gazebo reference="horn_2_link">
+      <material>Gazebo/White</material>
+    </gazebo>
   </xacro:macro>
 </robot>

Commit message: palm

File: hand_robot_ws/src/hand_description/urdf/hand.xacro (robot description, xacro)
@@ -17,5 +17,5 @@
   </xacro:wrist>
   <xacro:palm parent="wrist_link">
-    <origin xyz="0.041 -0.035 0.001" rpy="0 0 0"/>
+    <origin xyz="0.041 -0.033 0.001" rpy="${-90 * pi / 180} 0 0"/>
   </xacro:palm>
   <!-- ros2_control configuration -->

File: hand_robot_ws/src/hand_description/urdf/palm.xacro (robot description, xacro)
@@ -4,58 +4,8 @@
   <xacro:macro name="palm" params="parent *origin">
     <!-- Joint entre wrist et palm -->
-    <joint name="wrist_palm_joint" type="revolute">
+    <joint name="wrist_horn_joint" type="fixed">
       <parent link="${parent}"/>
-      <child link="palm_link"/>
-      <axis xyz="0 1 0"/>
-      <limit effort="10.0" lower="${-90 * pi / 180}" upper="${90 * pi / 180}" velocity="0.3"/>
+      <child link="horn_2_link"/>
       <xacro:insert_block name="origin"/>
-    </joint>
-    <!-- middle base left -->
-    <link name="palm_link">
-      <visual>
-        <geometry>
-          <mesh filename="package://hand_description/meshes/palm.stl" scale="0.001 0.001 0.001"/>
-        </geometry>
-        <material name="white"/>
-        <origin xyz="-0.022 0.02 0.004" rpy="${90 * pi / 180} ${-153 * pi / 180} ${95.5 * pi / 180}"/>
-      </visual>
-      <collision>
-        <geometry>
-          <mesh filename="package://hand_description/meshes/palm.stl" scale="0.001 0.001 0.001"/>
-        </geometry>
-        <origin xyz="0 0 0" rpy="0 0 0"/>
-      </collision>
-      <xacro:cylinder_inertia mass="0.5" radius="0.08" length="0.25"/>
-    </link>
-    <!-- Joint entre palm et servo -->
-    <joint name="palm_servo_joint" type="fixed">
-      <parent link="palm_link"/>
-      <child link="servo_2_link"/>
-      <origin xyz="0.01 0.047 0.001" rpy="${90 * pi / 180} ${180 * pi / 180} ${0 * pi / 180}"/>
-    </joint>
-    <!-- Servo link -->
-    <link name="servo_2_link">
-      <visual>
-        <geometry>
-          <mesh filename="package://hand_description/meshes/Servo_Hitec_HS_645MG.stl" scale="0.001 0.001 0.001"/>
-        </geometry>
-        <material name="black"/>
-        <origin xyz="0 0 0" rpy="0 0 0"/>
-      </visual>
-      <collision>
-        <geometry>
-          <mesh filename="package://hand_description/meshes/Servo_Hitec_HS_645MG.stl" scale="0.001 0.001 0.001"/>
-        </geometry>
-        <origin xyz="0 0 0" rpy="0 0 0"/>
-      </collision>
-      <xacro:cylinder_inertia mass="0.1" radius="0.02" length="0.04"/>
-    </link>
-    <!-- Joint entre servo et horn (revolute pour rotation)-->
-    <joint name="servo_horn_2_joint" type="revolute">
-      <parent link="servo_2_link"/>
-      <child link="horn_2_link"/>
-      <origin xyz="0.01 0 0.045" rpy="${180 * pi / 180} 0 0"/>
-      <axis xyz="0 0 1"/>
-      <limit effort="10.0" lower="${-180 * pi / 180}" upper="${180 * pi / 180}" velocity="0.3"/>
     </joint>
     <!-- Servo link -->
@@ -80,4 +30,52 @@
       <material>Gazebo/White</material>
     </gazebo>
+    <!-- Joint entre servo et horn (revolute pour rotation)-->
+    <joint name="servo_horn_2_joint" type="revolute">
+      <parent link="horn_2_link"/>
+      <child link="servo_2_link"/>
+      <origin xyz="0 0 0" rpy="0 0 0"/>
+      <axis xyz="0 0 1"/>
+      <limit effort="10.0" lower="${-90 * pi / 180}" upper="${90 * pi / 180}" velocity="0.3"/>
+    </joint>
+    <!-- Servo link -->
+    <link name="servo_2_link">
+      <visual>
+        <geometry>
+          <mesh filename="package://hand_description/meshes/Servo_Hitec_HS_645MG.stl" scale="0.001 0.001 0.001"/>
+        </geometry>
+        <material name="black"/>
+        <origin xyz="0.01 0 0.045" rpy="${180 * pi / 180} 0 ${180 * pi / 180}"/>
+      </visual>
+      <collision>
+        <geometry>
+          <mesh filename="package://hand_description/meshes/Servo_Hitec_HS_645MG.stl" scale="0.001 0.001 0.001"/>
+        </geometry>
+        <origin xyz="0 0 0" rpy="0 0 0"/>
+      </collision>
+      <xacro:cylinder_inertia mass="0.1" radius="0.02" length="0.04"/>
+    </link>
+    <!-- Joint entre palm et servo -->
+    <joint name="palm_servo_joint" type="fixed">
+      <parent link="servo_2_link"/>
+      <child link="palm_link"/>
+      <origin xyz="0 0 0" rpy="${90 * pi / 180} 0 0"/>
+    </joint>
+    <!-- middle base left -->
+    <link name="palm_link">
+      <visual>
+        <geometry>
+          <mesh filename="package://hand_description/meshes/palm.stl" scale="0.001 0.001 0.001"/>
+        </geometry>
+        <material name="white"/>
+        <origin xyz="-0.022 0.018 0.004" rpy="${90 * pi / 180} ${-153 * pi / 180} ${95.5 * pi / 180}"/>
+      </visual>
+      <collision>
+        <geometry>
+          <mesh filename="package://hand_description/meshes/palm.stl" scale="0.001 0.001 0.001"/>
+        </geometry>
+        <origin xyz="0 0 0" rpy="0 0 0"/>
+      </collision>
+      <xacro:cylinder_inertia mass="0.5" radius="0.08" length="0.25"/>
+    </link>
   </xacro:macro>
 </robot>
