Commit message: rod+steering_index_middle_ring

File: hand_robot_ws/src/hand_description/urdf/hand.xacro (robot description, xacro)
@@ -19,9 +19,9 @@
     <origin xyz="0.041 -0.033 0.001" rpy="${-90 * pi / 180} 0 0"/>
   </xacro:palm>
-  <!-- ros2_control configuration -->
-  <xacro:hand_ros2_control name="HandController" initial_positions_file=""/>
   <!-- <xacro:index parent="palm_link">
     <origin xyz="0 0.03 0.15" rpy="0 0 ${180 * pi / 180}"/>
   </xacro:index> -->
+  <!-- ros2_control configuration -->
+  <xacro:hand_ros2_control name="HandController" initial_positions_file=""/>
   <!-- <xacro:middle parent="base_footprint">
     <origin xyz="0 0.03 0" rpy="0 0 0"/>

File: hand_robot_ws/src/hand_description/urdf/palm.xacro (robot description, xacro)
@@ -107,5 +107,5 @@
       <origin xyz="0.0028 0.006 0.03" rpy="${-3 * pi / 180} ${10 * pi / 180} ${2 * pi / 180}"/>
       <axis xyz="0 0 1"/>
-      <limit effort="10.0" lower="${-70 * pi / 180}" upper="${50 * pi / 180}" velocity="0.3"/>
+      <limit effort="10.0" lower="${20 * pi / 180}" upper="${-10 * pi / 180}" velocity="0.3"/>
     </joint>
     <!-- middle base left -->
@@ -121,4 +121,76 @@
         <geometry>
           <mesh filename="package://hand_description/meshes/SG90_arm.stl" scale="0.001 0.001 0.001"/>
+        </geometry>
+        <origin xyz="0 0 0" rpy="0 0 0"/>
+      </collision>
+      <xacro:cylinder_inertia mass="0.5" radius="0.08" length="0.25"/>
+    </link>
+    <!-- Joint entre palm et servo -->
+    <joint name="arm_steering_index_joint" type="revolute">
+      <parent link="sg90_arm_index_link"/>
+      <child link="steering_index_link"/>
+      <origin xyz="0.01 0.0 0.0" rpy="${0 * pi / 180} ${0 * pi / 180} ${-90 * pi / 180}"/>
+      <axis xyz="0 0 1"/>
+      <limit effort="10.0" lower="${25 * pi / 180}" upper="${0 * pi / 180}" velocity="0.3"/>
+      <mimic joint="sg90_arm_index_joint" multiplier="-1" offset="${20 * pi / 180}"/>
+    </joint>
+    <!-- middle base left -->
+    <link name="steering_index_link">
+      <visual>
+        <geometry>
+          <mesh filename="package://hand_description/meshes/steeringlink_end_v2.stl" scale="0.001 0.001 0.001"/>
+        </geometry>
+        <material name="blue"/>
+        <origin xyz="0.003 0 0" rpy="${0 * pi / 180} ${0 * pi / 180} ${0 * pi / 180}"/>
+      </visual>
+      <collision>
+        <geometry>
+          <mesh filename="package://hand_description/meshes/steeringlink_end_v2.stl" scale="0.001 0.001 0.001"/>
+        </geometry>
+        <origin xyz="0 0 0" rpy="0 0 0"/>
+      </collision>
+      <xacro:cylinder_inertia mass="0.5" radius="0.08" length="0.25"/>
+    </link>
+    <!-- Joint entre palm et servo -->
+    <joint name="steering_rod_index_joint" type="fixed">
+      <parent link="steering_index_link"/>
+      <child link="rod_index_link"/>
+      <origin xyz="0.009 0.0 0.002" rpy="${0 * pi / 180} ${90 * pi / 180} ${0 * pi / 180}"/>
+    </joint>
+    <!-- middle base left -->
+    <link name="rod_index_link">
+      <visual>
+        <geometry>
+          <cylinder length="0.02" radius="0.0009"/>
+        </geometry>
+        <material name="gray"/>
+        <origin xyz="0.0 0 0.01" rpy="${0 * pi / 180} ${0 * pi / 180} ${0 * pi / 180}"/>
+      </visual>
+      <collision>
+        <geometry>
+            <cylinder length="0.02" radius="0.0009"/>
+        </geometry>
+        <origin xyz="0 0 0" rpy="0 0 0"/>
+      </collision>
+      <xacro:cylinder_inertia mass="0.5" radius="0.08" length="0.25"/>
+    </link>
+    <!-- Joint entre palm et servo -->
+    <joint name="steering_rod_end_index_joint" type="fixed">
+      <parent link="rod_index_link"/>
+      <child link="steering_end_index_link"/>
+      <origin xyz="0.0 0.0 0.02" rpy="${-90 * pi / 180} ${90 * pi / 180} ${0 * pi / 180}"/>
+    </joint>
+    <!-- middle base left -->
+    <link name="steering_end_index_link">
+      <visual>
+        <geometry>
+          <mesh filename="package://hand_description/meshes/steeringlink_end_v2.stl" scale="0.001 0.001 0.001"/>
+        </geometry>
+        <material name="blue"/>
+        <origin xyz="0.0 0 -0.002" rpy="${0 * pi / 180} ${0 * pi / 180} ${0 * pi / 180}"/>
+      </visual>
+      <collision>
+        <geometry>
+          <mesh filename="package://hand_description/meshes/steeringlink_end_v2.stl" scale="0.001 0.001 0.001"/>
         </geometry>
         <origin xyz="0 0 0" rpy="0 0 0"/>
@@ -155,5 +227,5 @@
       <origin xyz="0.0028 0.006 0.03" rpy="${-3 * pi / 180} ${10 * pi / 180} ${2 * pi / 180}"/>
       <axis xyz="0 0 1"/>
-      <limit effort="10.0" lower="${-70 * pi / 180}" upper="${50 * pi / 180}" velocity="0.3"/>
+      <limit effort="10.0" lower="${20 * pi / 180}" upper="${-10 * pi / 180}" velocity="0.3"/>
     </joint>
     <!-- middle base left -->
@@ -169,4 +241,76 @@
         <geometry>
           <mesh filename="package://hand_description/meshes/SG90_arm.stl" scale="0.001 0.001 0.001"/>
+        </geometry>
+        <origin xyz="0 0 0" rpy="0 0 0"/>
+      </collision>
+      <xacro:cylinder_inertia mass="0.5" radius="0.08" length="0.25"/>
+    </link>
+    <!-- Joint entre palm et servo -->
+    <joint name="arm_steering_middle_joint" type="revolute">
+      <parent link="sg90_arm_middle_link"/>
+      <child link="steering_middle_link"/>
+      <origin xyz="0.01 0.0 0.0" rpy="${0 * pi / 180} ${0 * pi / 180} ${-90 * pi / 180}"/>
+      <axis xyz="0 0 1"/>
+      <limit effort="10.0" lower="${25 * pi / 180}" upper="${0 * pi / 180}" velocity="0.3"/>
+      <mimic joint="sg90_arm_middle_joint" multiplier="-1" offset="${20 * pi / 180}"/>
+    </joint>
+    <!-- middle base left -->
+    <link name="steering_middle_link">
+      <visual>
+        <geometry>
+          <mesh filename="package://hand_description/meshes/steeringlink_end_v2.stl" scale="0.001 0.001 0.001"/>
+        </geometry>
+        <material name="blue"/>
+        <origin xyz="0.003 0 0" rpy="${0 * pi / 180} ${0 * pi / 180} ${0 * pi / 180}"/>
+      </visual>
+      <collision>
+        <geometry>
+          <mesh filename="package://hand_description/meshes/steeringlink_end_v2.stl" scale="0.001 0.001 0.001"/>
+        </geometry>
+        <origin xyz="0 0 0" rpy="0 0 0"/>
+      </collision>
+      <xacro:cylinder_inertia mass="0.5" radius="0.08" length="0.25"/>
+    </link>
+    <!-- Joint entre palm et servo -->
+    <joint name="steering_rod_middle_joint" type="fixed">
+      <parent link="steering_middle_link"/>
+      <child link="rod_middle_link"/>
+      <origin xyz="0.009 0.0 0.002" rpy="${0 * pi / 180} ${90 * pi / 180} ${0 * pi / 180}"/>
+    </joint>
+    <!-- middle base left -->
+    <link name="rod_middle_link">
+      <visual>
+        <geometry>
+          <cylinder length="0.02" radius="0.0009"/>
+        </geometry>
+        <material name="gray"/>
+        <origin xyz="0.0 0 0.01" rpy="${0 * pi / 180} ${0 * pi / 180} ${0 * pi / 180}"/>
+      </visual>
+      <collision>
+        <geometry>
+            <cylinder length="0.02" radius="0.0009"/>
+        </geometry>
+        <origin xyz="0 0 0" rpy="0 0 0"/>
+      </collision>
+      <xacro:cylinder_inertia mass="0.5" radius="0.08" length="0.25"/>
+    </link>
+    <!-- Joint entre palm et servo -->
+    <joint name="steering_rod_end_middle_joint" type="fixed">
+      <parent link="rod_middle_link"/>
+      <child link="steering_end_middle_link"/>
+      <origin xyz="0.0 0.0 0.02" rpy="${-90 * pi / 180} ${90 * pi / 180} ${0 * pi / 180}"/>
+    </joint>
+    <!-- middle base left -->
+    <link name="steering_end_middle_link">
+      <visual>
+        <geometry>
+          <mesh filename="package://hand_description/meshes/steeringlink_end_v2.stl" scale="0.001 0.001 0.001"/>
+        </geometry>
+        <material name="blue"/>
+        <origin xyz="0.0 0 -0.002" rpy="${0 * pi / 180} ${0 * pi / 180} ${0 * pi / 180}"/>
+      </visual>
+      <collision>
+        <geometry>
+          <mesh filename="package://hand_description/meshes/steeringlink_end_v2.stl" scale="0.001 0.001 0.001"/>
         </geometry>
         <origin xyz="0 0 0" rpy="0 0 0"/>
@@ -203,5 +347,5 @@
       <origin xyz="0.0028 0.006 0.03" rpy="${-3 * pi / 180} ${10 * pi / 180} ${2 * pi / 180}"/>
       <axis xyz="0 0 1"/>
-      <limit effort="10.0" lower="${-70 * pi / 180}" upper="${50 * pi / 180}" velocity="0.3"/>
+      <limit effort="10.0" lower="${20 * pi / 180}" upper="${-10 * pi / 180}" velocity="0.3"/>
     </joint>
     <!-- middle base left -->
@@ -217,4 +361,76 @@
         <geometry>
           <mesh filename="package://hand_description/meshes/SG90_arm.stl" scale="0.001 0.001 0.001"/>
+        </geometry>
+        <origin xyz="0 0 0" rpy="0 0 0"/>
+      </collision>
+      <xacro:cylinder_inertia mass="0.5" radius="0.08" length="0.25"/>
+    </link>
+    <!-- Joint entre palm et servo -->
+    <joint name="arm_steering_ring_joint" type="revolute">
+      <parent link="sg90_arm_ring_link"/>
+      <child link="steering_ring_link"/>
+      <origin xyz="0.01 0.0 0.0" rpy="${0 * pi / 180} ${0 * pi / 180} ${-90 * pi / 180}"/>
+      <axis xyz="0 0 1"/>
+      <limit effort="10.0" lower="${25 * pi / 180}" upper="${0 * pi / 180}" velocity="0.3"/>
+      <mimic joint="sg90_arm_ring_joint" multiplier="-1" offset="${20 * pi / 180}"/>
+    </joint>
+    <!-- middle base left -->
+    <link name="steering_ring_link">
+      <visual>
+        <geometry>
+          <mesh filename="package://hand_description/meshes/steeringlink_end_v2.stl" scale="0.001 0.001 0.001"/>
+        </geometry>
+        <material name="blue"/>
+        <origin xyz="0.003 0 0" rpy="${0 * pi / 180} ${0 * pi / 180} ${0 * pi / 180}"/>
+      </visual>
+      <collision>
+        <geometry>
+          <mesh filename="package://hand_description/meshes/steeringlink_end_v2.stl" scale="0.001 0.001 0.001"/>
+        </geometry>
+        <origin xyz="0 0 0" rpy="0 0 0"/>
+      </collision>
+      <xacro:cylinder_inertia mass="0.5" radius="0.08" length="0.25"/>
+    </link>
+    <!-- Joint entre palm et servo -->
+    <joint name="steering_rod_ring_joint" type="fixed">
+      <parent link="steering_ring_link"/>
+      <child link="rod_ring_link"/>
+      <origin xyz="0.009 0.0 0.002" rpy="${0 * pi / 180} ${90 * pi / 180} ${0 * pi / 180}"/>
+    </joint>
+    <!-- middle base left -->
+    <link name="rod_ring_link">
+      <visual>
+        <geometry>
+          <cylinder length="0.02" radius="0.0009"/>
+        </geometry>
+        <material name="gray"/>
+        <origin xyz="0.0 0 0.01" rpy="${0 * pi / 180} ${0 * pi / 180} ${0 * pi / 180}"/>
+      </visual>
+      <collision>
+        <geometry>
+            <cylinder length="0.02" radius="0.0009"/>
+        </geometry>
+        <origin xyz="0 0 0" rpy="0 0 0"/>
+      </collision>
+      <xacro:cylinder_inertia mass="0.5" radius="0.08" length="0.25"/>
+    </link>
+    <!-- Joint entre palm et servo -->
+    <joint name="steering_rod_end_ring_joint" type="fixed">
+      <parent link="rod_ring_link"/>
+      <child link="steering_end_ring_link"/>
+      <origin xyz="0.0 0.0 0.02" rpy="${-90 * pi / 180} ${90 * pi / 180} ${0 * pi / 180}"/>
+    </joint>
+    <!-- middle base left -->
+    <link name="steering_end_ring_link">
+      <visual>
+        <geometry>
+          <mesh filename="package://hand_description/meshes/steeringlink_end_v2.stl" scale="0.001 0.001 0.001"/>
+        </geometry>
+        <material name="blue"/>
+        <origin xyz="0.0 0 -0.002" rpy="${0 * pi / 180} ${0 * pi / 180} ${0 * pi / 180}"/>
+      </visual>
+      <collision>
+        <geometry>
+          <mesh filename="package://hand_description/meshes/steeringlink_end_v2.stl" scale="0.001 0.001 0.001"/>
         </geometry>
         <origin xyz="0 0 0" rpy="0 0 0"/>
@@ -251,5 +467,5 @@
       <origin xyz="0.0028 0.006 0.03" rpy="${-3 * pi / 180} ${10 * pi / 180} ${92 * pi / 180}"/>
       <axis xyz="0 0 1"/>
-      <limit effort="10.0" lower="${-70 * pi / 180}" upper="${30 * pi / 180}" velocity="0.3"/>
+      <limit effort="10.0" lower="${20 * pi / 180}" upper="${-10 * pi / 180}" velocity="0.3"/>
     </joint>
     <!-- middle base left -->

Commit message: finger_not_ok

File: hand_robot_ws/src/hand_description/urdf/hand.xacro (robot description, xacro)
@@ -7,5 +7,5 @@
   <xacro:include filename="$(find hand_description)/urdf/wrist.xacro"/>
   <xacro:include filename="$(find hand_description)/urdf/palm.xacro"/>
-  <!-- <xacro:include filename="$(find hand_description)/urdf/index.xacro"/> -->
+  <xacro:include filename="$(find hand_description)/urdf/index.xacro"/>
   <!-- <xacro:include filename="$(find hand_description)/urdf/middle.xacro"/> -->
   <link name="base_footprint"></link>
@@ -19,7 +19,8 @@
     <origin xyz="0.041 -0.033 0.001" rpy="${-90 * pi / 180} 0 0"/>
   </xacro:palm>
-  <!-- <xacro:index parent="palm_link">
-    <origin xyz="0 0.03 0.15" rpy="0 0 ${180 * pi / 180}"/>
-  </xacro:index> -->
+  <xacro:index parent="palm_link">
+    <origin xyz="-0.011 -0.018 0.0" rpy="${-90 * pi / 180} 0 ${0 * pi / 180}"/>
+    <mimic joint="sg90_arm_index_joint" multiplier="1" offset="${-20 * pi / 180}"/>
+  </xacro:index>
   <!-- ros2_control configuration -->
   <xacro:hand_ros2_control name="HandController" initial_positions_file=""/>

File: hand_robot_ws/src/hand_description/urdf/index.xacro (robot description, xacro)
@@ -2,10 +2,13 @@
 <robot xmlns:xacro="http://www.ros.org/wiki/xacro">
   <!-- Index of the hand -->
-  <xacro:macro name="index" params="parent *origin">
+  <xacro:macro name="index" params="parent *origin *mimic">
     <!-- Joint entre base_footprint et base_link -->
-    <joint name="index_base_joint_fixed" type="fixed">
+    <joint name="index_base_joint_fixed" type="revolute">
       <parent link="${parent}"/>
       <child link="index_base_left_link"/>
       <xacro:insert_block name="origin"/>
+      <axis xyz="0 1 0"/>
+      <limit effort="10.0" lower="${-30 * pi / 180}" upper="${0 * pi / 180}" velocity="0.3"/>
+      <xacro:insert_block name="mimic"/>
     </joint>
     <!-- index base left -->
@@ -16,5 +19,5 @@
         </geometry>
         <material name="white"/>
-        <origin xyz="0 0 0" rpy="0 0 0"/>
+        <origin xyz="0.004 -0.0148 -0.005" rpy="0 0 0"/>
       </visual>
       <collision>
@@ -27,15 +30,15 @@
     </link>
     <!-- Color Gazebo for index base left -->
-    <gazebo reference="index_base_left_link">
+    <!-- <gazebo reference="index_base_left_link">
       <material>Gazebo/White</material>
-    </gazebo>
-    <joint name="index_base_joint" type="prismatic">
+    </gazebo> -->
+    <!-- <joint name="index_base_joint" type="prismatic">
       <origin xyz="-0.03 0.014 0.01" rpy="${-90 * pi / 180} ${30 * pi / 180} 0"/>
       <parent link="index_base_left_link"/>
       <child link="index_base_right_link"/>
       <limit effort="1000.0" lower="0.002" upper="-0.004" velocity="0.8"/>
-    </joint>
+    </joint> -->
     <!-- index base right -->
-    <link name="index_base_right_link">
+    <!-- <link name="index_base_right_link">
       <visual>
         <geometry>
@@ -52,10 +55,10 @@
       </collision>
       <xacro:cylinder_inertia mass="0.5" radius="0.08" length="0.25"/>
-    </link>
+    </link> -->
     <!-- Color Gazebo for index base right -->
-    <gazebo reference="index_base_right_link">
+    <!-- <gazebo reference="index_base_right_link">
       <material>Gazebo/White</material>
-    </gazebo>
-    <joint name="index_middle_left_base_left_joint" type="revolute">
+    </gazebo> -->
+    <!-- <joint name="index_middle_left_base_left_joint" type="revolute">
       <origin xyz="-0.0565 0.0095 0.012" rpy="${90 * pi / 180} ${45 * pi / 180} 0"/>
       <parent link="index_base_left_link"/>
@@ -64,7 +67,7 @@
       <limit effort="1000.0" lower="2" upper="0" velocity="0.8"/>
       <mimic joint="index_base_joint" multiplier="-200" offset="${60 * pi / 180}"/>
-    </joint>
+    </joint> -->
     <!-- index base right -->
-    <link name="index_middle_left_link">
+    <!-- <link name="index_middle_left_link">
       <visual>
         <geometry>
@@ -81,10 +84,10 @@
       </collision>
       <xacro:cylinder_inertia mass="0.5" radius="0.08" length="0.25"/>
-    </link>
+    </link> -->
     <!-- Color Gazebo for index base right -->
-    <gazebo reference="index_middle_left_link">
+    <!-- <gazebo reference="index_middle_left_link">
       <material>Gazebo/White</material>
-    </gazebo>
-    <joint name="index_middle_right_base_left_joint" type="revolute">
+    </gazebo> -->
+    <!-- <joint name="index_middle_right_base_left_joint" type="revolute">
       <origin xyz="-0.056 0.014 0.018" rpy="${-90 * pi / 180} ${90 * pi / 180} 0"/>
       <parent link="index_base_left_link"/>
@@ -93,7 +96,7 @@
       <limit effort="1000.0" lower="2" upper="0" velocity="0.8"/>
       <mimic joint="index_base_joint" multiplier="200" offset="${60 * pi / 180}"/>
-    </joint>
+    </joint> -->
     <!-- index base right -->
-    <link name="index_middle_right_link">
+    <!-- <link name="index_middle_right_link">
       <visual>
         <geometry>
@@ -110,10 +113,10 @@
       </collision>
       <xacro:cylinder_inertia mass="0.5" radius="0.08" length="0.25"/>
-    </link>
+    </link> -->
     <!-- Color Gazebo for index base right -->
-    <gazebo reference="index_middle_left_link">
+    <!-- <gazebo reference="index_middle_left_link">
       <material>Gazebo/White</material>
-    </gazebo>
-    <joint name="index_end_middle_left_joint" type="revolute">
+    </gazebo> -->
+    <!-- <joint name="index_end_middle_left_joint" type="revolute">
       <origin xyz="-0.031 0 -0.003" rpy="${90 * pi / 180} 0 ${180 * pi / 180}"/>
       <parent link="index_middle_left_link"/>
@@ -122,7 +125,7 @@
       <limit effort="1000.0" lower="2" upper="0" velocity="0.8"/>
       <mimic joint="index_base_joint" multiplier="-200" offset="${60 * pi / 180}"/>
-    </joint>
+    </joint> -->
     <!-- index base right -->
-    <link name="index_end_link">
+    <!-- <link name="index_end_link">
       <visual>
         <geometry>
@@ -139,9 +142,9 @@
       </collision>
       <xacro:cylinder_inertia mass="0.5" radius="0.08" length="0.25"/>
-    </link>
+    </link> -->
     <!-- Color Gazebo for index base right -->
-    <gazebo reference="index_middle_left_link">
+    <!-- <gazebo reference="index_middle_left_link">
       <material>Gazebo/White</material>
-    </gazebo>
+    </gazebo> -->
   </xacro:macro>
 </robot>

File: hand_robot_ws/src/hand_description/urdf/palm.xacro (robot description, xacro)
@@ -82,5 +82,5 @@
       <parent link="palm_link"/>
       <child link="sg90_index_link"/>
-      <origin xyz="0.077 0.002 0.0075" rpy="${180 * pi / 180} ${0 * pi / 180} ${-100 * pi / 180}"/>
+      <origin xyz="0.08 0.002 0.014" rpy="${170 * pi / 180} ${0 * pi / 180} ${-100 * pi / 180}"/>
     </joint>
     <!-- middle base left -->
@@ -132,6 +132,6 @@
       <origin xyz="0.01 0.0 0.0" rpy="${0 * pi / 180} ${0 * pi / 180} ${-90 * pi / 180}"/>
       <axis xyz="0 0 1"/>
-      <limit effort="10.0" lower="${25 * pi / 180}" upper="${0 * pi / 180}" velocity="0.3"/>
-      <mimic joint="sg90_arm_index_joint" multiplier="-1" offset="${20 * pi / 180}"/>
+      <limit effort="10.0" lower="${30 * pi / 180}" upper="${0 * pi / 180}" velocity="0.3"/>
+      <mimic joint="sg90_arm_index_joint" multiplier="-1" offset="${10 * pi / 180}"/>
     </joint>
     <!-- middle base left -->
@@ -162,12 +162,12 @@
       <visual>
         <geometry>
-          <cylinder length="0.02" radius="0.0009"/>
+          <cylinder length="0.018" radius="0.0009"/>
         </geometry>
         <material name="gray"/>
-        <origin xyz="0.0 0 0.01" rpy="${0 * pi / 180} ${0 * pi / 180} ${0 * pi / 180}"/>
-      </visual>
-      <collision>
-        <geometry>
-            <cylinder length="0.02" radius="0.0009"/>
+        <origin xyz="0.0 0 0.009" rpy="${0 * pi / 180} ${0 * pi / 180} ${0 * pi / 180}"/>
+      </visual>
+      <collision>
+        <geometry>
+            <cylinder length="0.018" radius="0.0009"/>
         </geometry>
         <origin xyz="0 0 0" rpy="0 0 0"/>
@@ -179,5 +179,5 @@
       <parent link="rod_index_link"/>
       <child link="steering_end_index_link"/>
-      <origin xyz="0.0 0.0 0.02" rpy="${-90 * pi / 180} ${90 * pi / 180} ${0 * pi / 180}"/>
+      <origin xyz="0.0 0.0 0.018" rpy="${-90 * pi / 180} ${90 * pi / 180} ${0 * pi / 180}"/>
     </joint>
     <!-- middle base left -->
