Commit message: index

File: hand_robot_ws/src/hand_description/urdf/hand.xacro (robot description, xacro)
@@ -20,5 +20,5 @@
   </xacro:palm>
   <xacro:index parent="palm_link">
-    <origin xyz="-0.011 -0.018 0.0" rpy="${-90 * pi / 180} 0 ${0 * pi / 180}"/>
+    <origin xyz="0.104 -0.0206 -0.004" rpy="${190 * pi / 180} ${0 * pi / 180} ${160 * pi / 180}"/>
     <mimic joint="sg90_arm_index_joint" multiplier="1" offset="${-20 * pi / 180}"/>
   </xacro:index>

File: hand_robot_ws/src/hand_description/urdf/index.xacro (robot description, xacro)
@@ -19,5 +19,5 @@
         </geometry>
         <material name="white"/>
-        <origin xyz="0.004 -0.0148 -0.005" rpy="0 0 0"/>
+        <origin xyz="0.004 -0.0148 -0.005" rpy="0 ${-1 * pi / 180} 0"/>
       </visual>
       <collision>
@@ -30,15 +30,17 @@
     </link>
     <!-- Color Gazebo for index base left -->
-    <!-- <gazebo reference="index_base_left_link">
+    <gazebo reference="index_base_left_link">
       <material>Gazebo/White</material>
-    </gazebo> -->
-    <!-- <joint name="index_base_joint" type="prismatic">
-      <origin xyz="-0.03 0.014 0.01" rpy="${-90 * pi / 180} ${30 * pi / 180} 0"/>
-      <parent link="index_base_left_link"/>
+    </gazebo>
+    <joint name="index_base_joint" type="revolute">
+      <origin xyz="0.102 -0.0202 0.005" rpy="${190 * pi / 180} ${-29 * pi / 180} ${155 * pi / 180}"/>
+      <parent link="${parent}"/>
       <child link="index_base_right_link"/>
+      <axis xyz="0 1 0"/>
       <limit effort="1000.0" lower="0.002" upper="-0.004" velocity="0.8"/>
-    </joint> -->
+      <xacro:insert_block name="mimic"/>
+    </joint>
     <!-- index base right -->
-    <!-- <link name="index_base_right_link">
+    <link name="index_base_right_link">
       <visual>
         <geometry>
@@ -46,5 +48,5 @@
         </geometry>
         <material name="white"/>
-        <origin xyz="-0.03 0.0205 0" rpy="0 0 0"/>
+        <origin xyz="-0.058 0.001 -0.0212" rpy="${-90 * pi / 180} 0 0"/>
       </visual>
       <collision>
@@ -55,19 +57,19 @@
       </collision>
       <xacro:cylinder_inertia mass="0.5" radius="0.08" length="0.25"/>
-    </link> -->
+    </link>
     <!-- Color Gazebo for index base right -->
-    <!-- <gazebo reference="index_base_right_link">
+    <gazebo reference="index_base_right_link">
       <material>Gazebo/White</material>
-    </gazebo> -->
-    <!-- <joint name="index_middle_left_base_left_joint" type="revolute">
-      <origin xyz="-0.0565 0.0095 0.012" rpy="${90 * pi / 180} ${45 * pi / 180} 0"/>
+    </gazebo>
+    <joint name="index_middle_left_base_left_joint" type="revolute">
+      <origin xyz="-0.052 -0.005 0.006" rpy="${90 * pi / 180} ${70 * pi / 180} 0"/>
       <parent link="index_base_left_link"/>
       <child link="index_middle_left_link"/>
       <axis xyz="0 0 1"/>
-      <limit effort="1000.0" lower="2" upper="0" velocity="0.8"/>
-      <mimic joint="index_base_joint" multiplier="-200" offset="${60 * pi / 180}"/>
-    </joint> -->
+      <limit effort="1000.0" lower="${0 * pi / 180}" upper="${130 * pi / 180}" velocity="0.8"/>
+      <mimic joint="index_base_joint" multiplier="-1.6" offset="${60 * pi / 180}"/>
+    </joint>
     <!-- index base right -->
-    <!-- <link name="index_middle_left_link">
+    <link name="index_middle_left_link">
       <visual>
         <geometry>
@@ -84,19 +86,19 @@
       </collision>
       <xacro:cylinder_inertia mass="0.5" radius="0.08" length="0.25"/>
-    </link> -->
+    </link>
     <!-- Color Gazebo for index base right -->
-    <!-- <gazebo reference="index_middle_left_link">
+    <gazebo reference="index_middle_left_link">
       <material>Gazebo/White</material>
-    </gazebo> -->
-    <!-- <joint name="index_middle_right_base_left_joint" type="revolute">
-      <origin xyz="-0.056 0.014 0.018" rpy="${-90 * pi / 180} ${90 * pi / 180} 0"/>
+    </gazebo>
+    <joint name="index_middle_right_base_left_joint" type="revolute">
+      <origin xyz="-0.0515 0.0005 0.012" rpy="${-90 * pi / 180} ${115 * pi / 180} 0"/>
       <parent link="index_base_left_link"/>
       <child link="index_middle_right_link"/>
       <axis xyz="0 0 1"/>
-      <limit effort="1000.0" lower="2" upper="0" velocity="0.8"/>
-      <mimic joint="index_base_joint" multiplier="200" offset="${60 * pi / 180}"/>
-    </joint> -->
+      <limit effort="1000.0" lower="${0 * pi / 180}" upper="${130 * pi / 180}" velocity="0.8"/>
+      <mimic joint="index_base_joint" multiplier="1.6" offset="${60 * pi / 180}"/>
+    </joint>
     <!-- index base right -->
-    <!-- <link name="index_middle_right_link">
+    <link name="index_middle_right_link">
       <visual>
         <geometry>
@@ -113,19 +115,19 @@
       </collision>
       <xacro:cylinder_inertia mass="0.5" radius="0.08" length="0.25"/>
-    </link> -->
+    </link>
     <!-- Color Gazebo for index base right -->
-    <!-- <gazebo reference="index_middle_left_link">
+    <gazebo reference="index_middle_left_link">
       <material>Gazebo/White</material>
-    </gazebo> -->
-    <!-- <joint name="index_end_middle_left_joint" type="revolute">
-      <origin xyz="-0.031 0 -0.003" rpy="${90 * pi / 180} 0 ${180 * pi / 180}"/>
+    </gazebo>
+    <joint name="index_end_middle_left_joint" type="revolute">
+      <origin xyz="-0.031 0 -0.003" rpy="${90 * pi / 180} ${0 * pi / 180} ${140 * pi / 180}"/>
       <parent link="index_middle_left_link"/>
       <child link="index_end_link"/>
       <axis xyz="0 1 0"/>
-      <limit effort="1000.0" lower="2" upper="0" velocity="0.8"/>
-      <mimic joint="index_base_joint" multiplier="-200" offset="${60 * pi / 180}"/>
-    </joint> -->
+      <limit effort="1000.0" lower="${0 * pi / 180}" upper="${80 * pi / 180}" velocity="0.8"/>
+      <mimic joint="index_base_joint" multiplier="-1.4" offset="${60 * pi / 180}"/>
+    </joint>
     <!-- index base right -->
-    <!-- <link name="index_end_link">
+    <link name="index_end_link">
       <visual>
         <geometry>
@@ -142,9 +144,9 @@
       </collision>
       <xacro:cylinder_inertia mass="0.5" radius="0.08" length="0.25"/>
-    </link> -->
+    </link>
     <!-- Color Gazebo for index base right -->
-    <!-- <gazebo reference="index_middle_left_link">
+    <gazebo reference="index_middle_left_link">
       <material>Gazebo/White</material>
-    </gazebo> -->
+    </gazebo>
   </xacro:macro>
 </robot>

File: hand_robot_ws/src/hand_description/urdf/palm.xacro (robot description, xacro)
@@ -107,5 +107,5 @@
       <origin xyz="0.0028 0.006 0.03" rpy="${-3 * pi / 180} ${10 * pi / 180} ${2 * pi / 180}"/>
       <axis xyz="0 0 1"/>
-      <limit effort="10.0" lower="${20 * pi / 180}" upper="${-10 * pi / 180}" velocity="0.3"/>
+      <limit effort="10.0" lower="${20 * pi / 180}" upper="${-40 * pi / 180}" velocity="0.3"/>
     </joint>
     <!-- middle base left -->
@@ -132,6 +132,6 @@
       <origin xyz="0.01 0.0 0.0" rpy="${0 * pi / 180} ${0 * pi / 180} ${-90 * pi / 180}"/>
       <axis xyz="0 0 1"/>
-      <limit effort="10.0" lower="${30 * pi / 180}" upper="${0 * pi / 180}" velocity="0.3"/>
-      <mimic joint="sg90_arm_index_joint" multiplier="-1" offset="${10 * pi / 180}"/>
+      <limit effort="10.0" lower="${30 * pi / 180}" upper="${-20 * pi / 180}" velocity="0.3"/>
+      <mimic joint="sg90_arm_index_joint" multiplier="-1.1" offset="${10 * pi / 180}"/>
     </joint>
     <!-- middle base left -->

Commit message: ring_finger

File: hand_robot_ws/src/hand_description/urdf/hand.xacro (robot description, xacro)
@@ -9,4 +9,5 @@
   <xacro:include filename="$(find hand_description)/urdf/index.xacro"/>
   <!-- <xacro:include filename="$(find hand_description)/urdf/middle.xacro"/> -->
+  <xacro:include filename="$(find hand_description)/urdf/ring_finger.xacro"/>
   <link name="base_footprint"></link>
   <xacro:forearm parent="base_footprint">
@@ -23,8 +24,13 @@
     <mimic joint="sg90_arm_index_joint" multiplier="1" offset="${-20 * pi / 180}"/>
   </xacro:index>
+  <!-- <xacro:middle parent="palm_link">
+    <origin xyz="0.116 0.042 -0.014" rpy="${190 * pi / 180} ${0 * pi / 180} ${180  * pi / 180}"/>
+    <mimic joint="sg90_arm_index_joint" multiplier="1" offset="${-20 * pi / 180}"/>
+  </xacro:middle> -->
+  <xacro:ring parent="palm_link">
+    <origin xyz="0.116 0.042 -0.014" rpy="${190 * pi / 180} ${0 * pi / 180} ${180 * pi / 180}"/>
+    <mimic joint="sg90_arm_ring_joint" multiplier="1" offset="${-20 * pi / 180}"/>
+  </xacro:ring>
   <!-- ros2_control configuration -->
   <xacro:hand_ros2_control name="HandController" initial_positions_file=""/>
-  <!-- <xacro:middle parent="base_footprint">
-    <origin xyz="0 0.03 0" rpy="0 0 0"/>
-  </xacro:middle> -->
 </robot>

File: hand_robot_ws/src/hand_description/urdf/palm.xacro (robot description, xacro)
@@ -347,5 +347,5 @@
       <origin xyz="0.0028 0.006 0.03" rpy="${-3 * pi / 180} ${10 * pi / 180} ${2 * pi / 180}"/>
       <axis xyz="0 0 1"/>
-      <limit effort="10.0" lower="${20 * pi / 180}" upper="${-10 * pi / 180}" velocity="0.3"/>
+      <limit effort="10.0" lower="${20 * pi / 180}" upper="${-40 * pi / 180}" velocity="0.3"/>
     </joint>
     <!-- middle base left -->

Commit message: middle_finger

File: hand_robot_ws/src/hand_description/urdf/hand.xacro (robot description, xacro)
@@ -7,7 +7,9 @@
   <xacro:include filename="$(find hand_description)/urdf/wrist.xacro"/>
   <xacro:include filename="$(find hand_description)/urdf/palm.xacro"/>
+  <!-- <xacro:include filename="$(find hand_description)/urdf/thumb.xacro"/> -->
   <xacro:include filename="$(find hand_description)/urdf/index.xacro"/>
-  <!-- <xacro:include filename="$(find hand_description)/urdf/middle.xacro"/> -->
+  <xacro:include filename="$(find hand_description)/urdf/middle_finger.xacro"/>
   <xacro:include filename="$(find hand_description)/urdf/ring_finger.xacro"/>
+  <!-- <xacro:include filename="$(find hand_description)/urdf/pinky_finger.xacro"/> -->
   <link name="base_footprint"></link>
   <xacro:forearm parent="base_footprint">
@@ -20,16 +22,25 @@
     <origin xyz="0.041 -0.033 0.001" rpy="${-90 * pi / 180} 0 0"/>
   </xacro:palm>
+  <!-- <xacro:thumb parent="palm_link">
+    <origin xyz="0.116 0.042 -0.014" rpy="${190 * pi / 180} ${0 * pi / 180} ${180  * pi / 180}"/>
+    <mimic joint="sg90_arm_thumb_joint" multiplier="1" offset="${-20 * pi / 180}"/>
+  </xacro:thumb> -->
   <xacro:index parent="palm_link">
     <origin xyz="0.104 -0.0206 -0.004" rpy="${190 * pi / 180} ${0 * pi / 180} ${160 * pi / 180}"/>
-    <mimic joint="sg90_arm_index_joint" multiplier="1" offset="${-20 * pi / 180}"/>
+    <mimic joint="sg90_arm_index_joint" multiplier="1.2" offset="${-20 * pi / 180}"/>
   </xacro:index>
-  <!-- <xacro:middle parent="palm_link">
+  <xacro:middle parent="palm_link">
+    <origin xyz="0.114 0.007 -0.011" rpy="${185 * pi / 180} ${0 * pi / 180} ${170  * pi / 180}"/>
+    <mimic joint="sg90_arm_middle_joint" multiplier="1.2" offset="${-20 * pi / 180}"/>
+  </xacro:middle>
+1
+  <xacro:ring parent="palm_link">
+    <origin xyz="0.116 0.0388 -0.014" rpy="${180 * pi / 180} ${0 * pi / 180} ${180 * pi / 180}"/>
+    <mimic joint="sg90_arm_ring_joint" multiplier="1.2" offset="${-20 * pi / 180}"/>
+  </xacro:ring>
+  <!-- <xacro:pinky parent="palm_link">
     <origin xyz="0.116 0.042 -0.014" rpy="${190 * pi / 180} ${0 * pi / 180} ${180  * pi / 180}"/>
-    <mimic joint="sg90_arm_index_joint" multiplier="1" offset="${-20 * pi / 180}"/>
-  </xacro:middle> -->
-  <xacro:ring parent="palm_link">
-    <origin xyz="0.116 0.042 -0.014" rpy="${190 * pi / 180} ${0 * pi / 180} ${180 * pi / 180}"/>
-    <mimic joint="sg90_arm_ring_joint" multiplier="1" offset="${-20 * pi / 180}"/>
-  </xacro:ring>
+    <mimic joint="sg90_arm_pinky_joint" multiplier="1" offset="${-20 * pi / 180}"/>
+  </xacro:pinky> -->
   <!-- ros2_control configuration -->
   <xacro:hand_ros2_control name="HandController" initial_positions_file=""/>

File: hand_robot_ws/src/hand_description/urdf/index.xacro (robot description, xacro)
@@ -92,5 +92,5 @@
     </gazebo>
     <joint name="index_middle_right_base_left_joint" type="revolute">
-      <origin xyz="-0.0515 0.0005 0.012" rpy="${-90 * pi / 180} ${115 * pi / 180} 0"/>
+      <origin xyz="-0.0515 -0.0005 0.012" rpy="${-90 * pi / 180} ${115 * pi / 180} 0"/>
       <parent link="index_base_left_link"/>
       <child link="index_middle_right_link"/>

File: hand_robot_ws/src/hand_description/urdf/middle_finger.xacro (robot description, xacro)
@@ -2,10 +2,13 @@
 <robot xmlns:xacro="http://www.ros.org/wiki/xacro">
   <!-- middle of the hand -->
-  <xacro:macro name="middle" params="parent *origin">
+  <xacro:macro name="middle" params="parent *origin *mimic">
     <!-- Joint entre base_footprint et base_link -->
-    <joint name="middle_base_joint_fixed" type="fixed">
+    <joint name="middle_base_joint_fixed" type="revolute">
       <parent link="${parent}"/>
       <child link="middle_base_left_link"/>
       <xacro:insert_block name="origin"/>
+      <axis xyz="0 1 0"/>
+      <limit effort="10.0" lower="${-30 * pi / 180}" upper="${0 * pi / 180}" velocity="0.3"/>
+      <xacro:insert_block name="mimic"/>
     </joint>
     <!-- middle base left -->
@@ -16,5 +19,5 @@
         </geometry>
         <material name="white"/>
-        <origin xyz="0.004 0.028 0" rpy="0 0 0"/>
+        <origin xyz="0.0085 0.014 -0.0055" rpy="0 0 0"/>
       </visual>
       <collision>
@@ -30,9 +33,11 @@
       <material>Gazebo/White</material>
     </gazebo>
-    <joint name="middle_base_joint" type="prismatic">
-      <origin xyz="-0.03 0.0147 0.01" rpy="${-90 * pi / 180} ${28 * pi / 180} 0"/>
-      <parent link="middle_base_left_link"/>
+    <joint name="middle_base_joint" type="revolute">
+      <origin xyz="0.111 0.0079 -0.001" rpy="${185 * pi / 180} ${-29 * pi / 180} ${167 * pi / 180}"/>
+      <parent link="${parent}"/>
       <child link="middle_base_right_link"/>
+      <axis xyz="0 1 0"/>
       <limit effort="1000.0" lower="0.002" upper="-0.004" velocity="0.8"/>
+      <xacro:insert_block name="mimic"/>
     </joint>
     <!-- middle base right -->
@@ -43,5 +48,5 @@
         </geometry>
         <material name="white"/>
-        <origin xyz="-0.03 -0.0209 0" rpy="0 0 0"/>
+        <origin xyz="-0.06 0.001 0.0212" rpy="${-90 * pi / 180} 0 0"/>
       </visual>
       <collision>
@@ -58,10 +63,10 @@
     </gazebo>
     <joint name="middle_middle_left_base_left_joint" type="revolute">
-      <origin xyz="-0.056 0.0103 0.0108" rpy="${90 * pi / 180} ${45 * pi / 180} 0"/>
+      <origin xyz="-0.0516 -0.0038 0.005" rpy="${90 * pi / 180} ${70 * pi / 180} 0"/>
       <parent link="middle_base_left_link"/>
       <child link="middle_middle_left_link"/>
       <axis xyz="0 0 1"/>
-      <limit effort="1000.0" lower="2" upper="0" velocity="0.8"/>
-      <mimic joint="middle_base_joint" multiplier="-200" offset="${60 * pi / 180}"/>
+      <limit effort="1000.0" lower="${0 * pi / 180}" upper="${130 * pi / 180}" velocity="0.8"/>
+      <mimic joint="middle_base_joint" multiplier="-1.6" offset="${60 * pi / 180}"/>
     </joint>
     <!-- middle base right -->
@@ -87,10 +92,10 @@
     </gazebo>
     <joint name="middle_middle_right_base_left_joint" type="revolute">
-      <origin xyz="-0.0555 0.0147 0.0167" rpy="${-90 * pi / 180} ${90 * pi / 180} 0"/>
+      <origin xyz="-0.0515 0.0009 0.012" rpy="${-90 * pi / 180} ${115 * pi / 180} 0"/>
       <parent link="middle_base_left_link"/>
       <child link="middle_middle_right_link"/>
       <axis xyz="0 0 1"/>
-      <limit effort="1000.0" lower="2" upper="0" velocity="0.8"/>
-      <mimic joint="middle_base_joint" multiplier="200" offset="${60 * pi / 180}"/>
+      <limit effort="1000.0" lower="${0 * pi / 180}" upper="${130 * pi / 180}" velocity="0.8"/>
+      <mimic joint="middle_base_joint" multiplier="1.6" offset="${60 * pi / 180}"/>
     </joint>
     <!-- middle base right -->
@@ -115,12 +120,12 @@
       <material>Gazebo/White</material>
     </gazebo>
-    <joint name="middle_end_middle_left_joint" type="revolute">
-      <origin xyz="-0.031 0 -0.003" rpy="${90 * pi / 180} 0 ${180 * pi / 180}"/>
-      <parent link="middle_middle_left_link"/>
-      <child link="middle_end_link"/>
-      <axis xyz="0 1 0"/>
-      <limit effort="1000.0" lower="2" upper="0" velocity="0.8"/>
-      <mimic joint="middle_base_joint" multiplier="-200" offset="${60 * pi / 180}"/>
-    </joint>
+      <joint name="middle_end_middle_left_joint" type="revolute">
+        <origin xyz="-0.0378 0 -0.003" rpy="${90 * pi / 180} 0 ${140 * pi / 180}"/>
+        <parent link="middle_middle_left_link"/>
+        <child link="middle_end_link"/>
+        <axis xyz="0 1 0"/>
+        <limit effort="1000.0" lower="${0 * pi / 180}" upper="${80 * pi / 180}" velocity="0.8"/>
+        <mimic joint="middle_base_joint" multiplier="-1.4" offset="${60 * pi / 180}"/>
+      </joint>
     <!-- middle base right -->
     <link name="middle_end_link">
@@ -130,5 +135,5 @@
         </geometry>
         <material name="white"/>
-        <origin xyz="-0.0241 -0.0156 -0.0058" rpy="0 0 0"/>
+        <origin xyz="0.041 -0.0156 -0.0058" rpy="0 0 0"/>
       </visual>
       <collision>

File: hand_robot_ws/src/hand_description/urdf/palm.xacro (robot description, xacro)
@@ -227,5 +227,5 @@
       <origin xyz="0.0028 0.006 0.03" rpy="${-3 * pi / 180} ${10 * pi / 180} ${2 * pi / 180}"/>
       <axis xyz="0 0 1"/>
-      <limit effort="10.0" lower="${20 * pi / 180}" upper="${-10 * pi / 180}" velocity="0.3"/>
+      <limit effort="10.0" lower="${20 * pi / 180}" upper="${-40 * pi / 180}" velocity="0.3"/>
     </joint>
     <!-- middle base left -->

File: hand_robot_ws/src/hand_description/urdf/ring_finger.xacro (robot description, xacro)
@@ -34,5 +34,5 @@
     </gazebo>
     <joint name="ring_base_joint" type="revolute">
-      <origin xyz="0.114 0.0424 -0.003" rpy="${190 * pi / 180} ${-29 * pi / 180} ${175 * pi / 180}"/>
+      <origin xyz="0.114 0.0374 -0.003" rpy="${180 * pi / 180} ${-29 * pi / 180} ${180 * pi / 180}"/>
       <parent link="${parent}"/>
       <child link="ring_base_right_link"/>
@@ -92,5 +92,5 @@
     </gazebo>
     <joint name="ring_middle_right_base_left_joint" type="revolute">
-      <origin xyz="-0.0515 0.0005 0.012" rpy="${-90 * pi / 180} ${115 * pi / 180} 0"/>
+      <origin xyz="-0.0515 -0.0005 0.012" rpy="${-90 * pi / 180} ${115 * pi / 180} 0"/>
       <parent link="ring_base_left_link"/>
       <child link="ring_middle_right_link"/>
