Commit message: thumb

File: hand_robot_ws/src/hand_description/urdf/hand.xacro (robot description, xacro)
@@ -7,5 +7,5 @@
   <xacro:include filename="$(find hand_description)/urdf/wrist.xacro"/>
   <xacro:include filename="$(find hand_description)/urdf/palm.xacro"/>
-  <!-- <xacro:include filename="$(find hand_description)/urdf/thumb.xacro"/> -->
+  <xacro:include filename="$(find hand_description)/urdf/thumb.xacro"/>
   <xacro:include filename="$(find hand_description)/urdf/index.xacro"/>
   <xacro:include filename="$(find hand_description)/urdf/middle_finger.xacro"/>
@@ -22,8 +22,8 @@
     <origin xyz="0.041 -0.033 0.001" rpy="${-90 * pi / 180} 0 0"/>
   </xacro:palm>
-  <!-- <xacro:thumb parent="palm_link">
-    <origin xyz="0.116 0.042 -0.014" rpy="${190 * pi / 180} ${0 * pi / 180} ${180  * pi / 180}"/>
-    <mimic joint="sg90_arm_thumb_joint" multiplier="1" offset="${-20 * pi / 180}"/>
-  </xacro:thumb> -->
+  <xacro:thumb parent="palm_link">
+    <origin xyz="0.057 -0.012 0.013" rpy="${180 * pi / 180} ${0 * pi / 180} ${55  * pi / 180}"/>
+    <mimic joint="sg90_arm_thumb_joint" multiplier="1" offset="${-100 * pi / 180}"/>
+  </xacro:thumb>
   <xacro:index parent="palm_link">
     <origin xyz="0.104 -0.0206 -0.004" rpy="${190 * pi / 180} ${0 * pi / 180} ${160 * pi / 180}"/>

File: hand_robot_ws/src/hand_description/urdf/palm.xacro (robot description, xacro)
@@ -79,4 +79,52 @@
     </link>
     <!-- Joint entre palm et servo -->
+    <joint name="palm_sg90_thumb_joint" type="fixed">
+      <parent link="palm_link"/>
+      <child link="sg90_thumb_link"/>
+      <origin xyz="0.051 0.015 0.007" rpy="${170 * pi / 180} ${10 * pi / 180} ${2 * pi / 180}"/>
+    </joint>
+    <!-- middle base left -->
+    <link name="sg90_thumb_link">
+      <visual>
+        <geometry>
+          <mesh filename="package://hand_description/meshes/SG90.stl" scale="0.001 0.001 0.001"/>
+        </geometry>
+        <material name="black"/>
+        <origin xyz="-0.0025 -0.001 0" rpy="${-3 * pi / 180} ${10 * pi / 180} ${2 * pi / 180}"/>
+      </visual>
+      <collision>
+        <geometry>
+          <mesh filename="package://hand_description/meshes/SG90.stl" scale="0.001 0.001 0.001"/>
+        </geometry>
+        <origin xyz="0 0 0" rpy="0 0 0"/>
+      </collision>
+      <xacro:cylinder_inertia mass="0.5" radius="0.08" length="0.25"/>
+    </link>
+    <!-- Joint entre palm et servo -->
+    <joint name="sg90_arm_thumb_joint" type="revolute">
+      <parent link="sg90_thumb_link"/>
+      <child link="sg90_arm_thumb_link"/>
+      <origin xyz="0.0028 0.006 0.03" rpy="${-3 * pi / 180} ${10 * pi / 180} ${182 * pi / 180}"/>
+      <axis xyz="0 0 1"/>
+      <limit effort="10.0" lower="${40 * pi / 180}" upper="${-10 * pi / 180}" velocity="0.3"/>
+    </joint>
+    <!-- middle base left -->
+    <link name="sg90_arm_thumb_link">
+      <visual>
+        <geometry>
+          <mesh filename="package://hand_description/meshes/SG90_arm.stl" scale="0.001 0.001 0.001"/>
+        </geometry>
+        <material name="orange"/>
+        <origin xyz="0.0067 0.0003 0" rpy="${180 * pi / 180} ${0 * pi / 180} ${90 * pi / 180}"/>
+      </visual>
+      <collision>
+        <geometry>
+          <mesh filename="package://hand_description/meshes/SG90_arm.stl" scale="0.001 0.001 0.001"/>
+        </geometry>
+        <origin xyz="0 0 0" rpy="0 0 0"/>
+      </collision>
+      <xacro:cylinder_inertia mass="0.5" radius="0.08" length="0.25"/>
+    </link>
+    <!-- Joint entre palm et servo -->
     <joint name="palm_sg90_index_joint" type="fixed">
       <parent link="palm_link"/>
@@ -486,52 +534,4 @@
       <xacro:cylinder_inertia mass="0.5" radius="0.08" length="0.25"/>
     </link>
-    <!-- Joint entre palm et servo -->
-    <joint name="palm_sg90_thumb_joint" type="fixed">
-      <parent link="palm_link"/>
-      <child link="sg90_thumb_link"/>
-      <origin xyz="0.051 0.015 0.007" rpy="${170 * pi / 180} ${10 * pi / 180} ${2 * pi / 180}"/>
-    </joint>
-    <!-- middle base left -->
-    <link name="sg90_thumb_link">
-      <visual>
-        <geometry>
-          <mesh filename="package://hand_description/meshes/SG90.stl" scale="0.001 0.001 0.001"/>
-        </geometry>
-        <material name="black"/>
-        <origin xyz="-0.0025 -0.001 0" rpy="${-3 * pi / 180} ${10 * pi / 180} ${2 * pi / 180}"/>
-      </visual>
-      <collision>
-        <geometry>
-          <mesh filename="package://hand_description/meshes/SG90.stl" scale="0.001 0.001 0.001"/>
-        </geometry>
-        <origin xyz="0 0 0" rpy="0 0 0"/>
-      </collision>
-      <xacro:cylinder_inertia mass="0.5" radius="0.08" length="0.25"/>
-    </link>
-    <!-- Joint entre palm et servo -->
-    <joint name="sg90_arm_thumb_joint" type="revolute">
-      <parent link="sg90_thumb_link"/>
-      <child link="sg90_arm_thumb_link"/>
-      <origin xyz="0.0028 0.006 0.03" rpy="${-3 * pi / 180} ${10 * pi / 180} ${92 * pi / 180}"/>
-      <axis xyz="0 0 1"/>
-      <limit effort="10.0" lower="${0 * pi / 180}" upper="${90 * pi / 180}" velocity="0.3"/>
-    </joint>
-    <!-- middle base left -->
-    <link name="sg90_arm_thumb_link">
-      <visual>
-        <geometry>
-          <mesh filename="package://hand_description/meshes/SG90_arm.stl" scale="0.001 0.001 0.001"/>
-        </geometry>
-        <material name="orange"/>
-        <origin xyz="0.0067 0.0003 0" rpy="${180 * pi / 180} ${0 * pi / 180} ${90 * pi / 180}"/>
-      </visual>
-      <collision>
-        <geometry>
-          <mesh filename="package://hand_description/meshes/SG90_arm.stl" scale="0.001 0.001 0.001"/>
-        </geometry>
-        <origin xyz="0 0 0" rpy="0 0 0"/>
-      </collision>
-      <xacro:cylinder_inertia mass="0.5" radius="0.08" length="0.25"/>
-    </link>
   </xacro:macro>
 </robot>

Commit message: pinky_base

File: hand_robot_ws/src/hand_description/urdf/hand.xacro (robot description, xacro)
@@ -11,5 +11,5 @@
   <xacro:include filename="$(find hand_description)/urdf/middle_finger.xacro"/>
   <xacro:include filename="$(find hand_description)/urdf/ring_finger.xacro"/>
-  <!-- <xacro:include filename="$(find hand_description)/urdf/pinky_finger.xacro"/> -->
+  <xacro:include filename="$(find hand_description)/urdf/pinky_finger.xacro"/>
   <link name="base_footprint"></link>
   <xacro:forearm parent="base_footprint">
@@ -39,8 +39,8 @@
     <mimic joint="sg90_arm_ring_joint" multiplier="1.2" offset="${-20 * pi / 180}"/>
   </xacro:ring>
-  <!-- <xacro:pinky parent="palm_link">
-    <origin xyz="0.116 0.042 -0.014" rpy="${190 * pi / 180} ${0 * pi / 180} ${180  * pi / 180}"/>
-    <mimic joint="sg90_arm_pinky_joint" multiplier="1" offset="${-20 * pi / 180}"/>
-  </xacro:pinky> -->
+  <xacro:pinky parent="palm_link">
+    <origin xyz="0.114 0.07 -0.015" rpy="${175 * pi / 180} ${0 * pi / 180} ${190 * pi / 180}"/>
+    <mimic joint="sg90_arm_pinky_joint" multiplier="-1" offset="${-20 * pi / 180}"/>
+  </xacro:pinky>
   <!-- ros2_control configuration -->
   <xacro:hand_ros2_control name="HandController" initial_positions_file=""/>

File: hand_robot_ws/src/hand_description/urdf/palm.xacro (robot description, xacro)
@@ -515,5 +515,5 @@
       <origin xyz="0.0028 0.006 0.03" rpy="${-3 * pi / 180} ${10 * pi / 180} ${92 * pi / 180}"/>
       <axis xyz="0 0 1"/>
-      <limit effort="10.0" lower="${20 * pi / 180}" upper="${-10 * pi / 180}" velocity="0.3"/>
+      <limit effort="10.0" lower="${-20 * pi / 180}" upper="${40 * pi / 180}" velocity="0.3"/>
     </joint>
     <!-- middle base left -->

File: hand_robot_ws/src/hand_description/urdf/pinky_finger.xacro (robot description, xacro)
@@ -19,5 +19,5 @@
         </geometry>
         <material name="white"/>
-        <origin xyz="0.004 -0.0148 -0.005" rpy="0 ${-1 * pi / 180} 0"/>
+        <origin xyz="-0.012 -0.0006 -0.005" rpy="0 ${-1 * pi / 180} ${180 * pi / 180}"/>
       </visual>
       <collision>
@@ -34,5 +34,5 @@
     </gazebo>
     <joint name="pinky_base_joint" type="revolute">
-      <origin xyz="0.114 0.0374 -0.003" rpy="${180 * pi / 180} ${-29 * pi / 180} ${180 * pi / 180}"/>
+      <origin xyz="0.111 0.067 -0.005" rpy="${175 * pi / 180} ${-40 * pi / 180} ${195 * pi / 180}"/>
       <parent link="${parent}"/>
       <child link="pinky_base_right_link"/>
@@ -48,5 +48,5 @@
         </geometry>
         <material name="white"/>
-        <origin xyz="-0.058 0.001 -0.0212" rpy="${-90 * pi / 180} 0 0"/>
+        <origin xyz="-0.016 0.001 -0.0" rpy="${-90 * pi / 180} 0 0"/>
       </visual>
       <collision>
@@ -62,5 +62,5 @@
       <material>Gazebo/White</material>
     </gazebo>
-    <joint name="pinky_middle_left_base_left_joint" type="revolute">
+    <!-- <joint name="pinky_middle_left_base_left_joint" type="revolute">
       <origin xyz="-0.052 -0.005 0.006" rpy="${90 * pi / 180} ${70 * pi / 180} 0"/>
       <parent link="pinky_base_left_link"/>
@@ -69,7 +69,7 @@
       <limit effort="1000.0" lower="${0 * pi / 180}" upper="${130 * pi / 180}" velocity="0.8"/>
       <mimic joint="pinky_base_joint" multiplier="-1.6" offset="${60 * pi / 180}"/>
-    </joint>
+    </joint> -->
     <!-- pinky base right -->
-    <link name="pinky_middle_left_link">
+    <!-- <link name="pinky_middle_left_link">
       <visual>
         <geometry>
@@ -86,10 +86,10 @@
       </collision>
       <xacro:cylinder_inertia mass="0.5" radius="0.08" length="0.25"/>
-    </link>
+    </link>  -->
     <!-- Color Gazebo for pinky base right -->
-    <gazebo reference="pinky_middle_left_link">
+    <!-- <gazebo reference="pinky_middle_left_link">
       <material>Gazebo/White</material>
-    </gazebo>
-    <joint name="pinky_middle_right_base_left_joint" type="revolute">
+    </gazebo> -->
+    <!-- <joint name="pinky_middle_right_base_left_joint" type="revolute">
       <origin xyz="-0.0515 -0.0005 0.012" rpy="${-90 * pi / 180} ${115 * pi / 180} 0"/>
       <parent link="pinky_base_left_link"/>
@@ -98,7 +98,7 @@
       <limit effort="1000.0" lower="${0 * pi / 180}" upper="${130 * pi / 180}" velocity="0.8"/>
       <mimic joint="pinky_base_joint" multiplier="1.6" offset="${60 * pi / 180}"/>
-    </joint>
+    </joint> -->
     <!-- pinky base right -->
-    <link name="pinky_middle_right_link">
+    <!-- <link name="pinky_middle_right_link">
       <visual>
         <geometry>
@@ -115,10 +115,10 @@
       </collision>
       <xacro:cylinder_inertia mass="0.5" radius="0.08" length="0.25"/>
-    </link>
+    </link> -->
     <!-- Color Gazebo for pinky base right -->
-    <gazebo reference="pinky_middle_left_link">
+    <!-- <gazebo reference="pinky_middle_left_link">
       <material>Gazebo/White</material>
-    </gazebo>
-    <joint name="pinky_end_middle_left_joint" type="revolute">
+    </gazebo> -->
+    <!-- <joint name="pinky_end_middle_left_joint" type="revolute">
       <origin xyz="-0.031 0 -0.003" rpy="${90 * pi / 180} ${0 * pi / 180} ${140 * pi / 180}"/>
       <parent link="pinky_middle_left_link"/>
@@ -127,7 +127,7 @@
       <limit effort="1000.0" lower="${0 * pi / 180}" upper="${80 * pi / 180}" velocity="0.8"/>
       <mimic joint="pinky_base_joint" multiplier="-1.4" offset="${60 * pi / 180}"/>
-    </joint>
+    </joint> -->
     <!-- pinky base right -->
-    <link name="pinky_end_link">
+    <!-- <link name="pinky_end_link">
       <visual>
         <geometry>
@@ -144,9 +144,9 @@
       </collision>
       <xacro:cylinder_inertia mass="0.5" radius="0.08" length="0.25"/>
-    </link>
+    </link> -->
     <!-- Color Gazebo for pinky base right -->
-    <gazebo reference="pinky_middle_left_link">
+    <!-- <gazebo reference="pinky_middle_left_link">
       <material>Gazebo/White</material>
-    </gazebo>
+    </gazebo> -->
   </xacro:macro>
 </robot>

Commit message: pinky_ok

File: hand_robot_ws/src/hand_description/urdf/hand.xacro (robot description, xacro)
@@ -14,5 +14,5 @@
   <link name="base_footprint"></link>
   <xacro:forearm parent="base_footprint">
-    <origin xyz="0 0 0" rpy="0 0 0"/>
+    <origin xyz="0 0 0" rpy="0 ${90 * pi / 180} 0"/>
   </xacro:forearm>
   <xacro:wrist parent="horn_link">
@@ -41,5 +41,5 @@
   <xacro:pinky parent="palm_link">
     <origin xyz="0.114 0.07 -0.015" rpy="${175 * pi / 180} ${0 * pi / 180} ${190 * pi / 180}"/>
-    <mimic joint="sg90_arm_pinky_joint" multiplier="-1" offset="${-20 * pi / 180}"/>
+    <mimic joint="sg90_arm_pinky_joint" multiplier="-1.2" offset="${-20 * pi / 180}"/>
   </xacro:pinky>
   <!-- ros2_control configuration -->

File: hand_robot_ws/src/hand_description/urdf/index.xacro (robot description, xacro)
@@ -68,5 +68,5 @@
       <axis xyz="0 0 1"/>
       <limit effort="1000.0" lower="${0 * pi / 180}" upper="${130 * pi / 180}" velocity="0.8"/>
-      <mimic joint="index_base_joint" multiplier="-1.6" offset="${60 * pi / 180}"/>
+      <mimic joint="index_base_joint" multiplier="-1.4" offset="${60 * pi / 180}"/>
     </joint>
     <!-- index base right -->
@@ -97,5 +97,5 @@
       <axis xyz="0 0 1"/>
       <limit effort="1000.0" lower="${0 * pi / 180}" upper="${130 * pi / 180}" velocity="0.8"/>
-      <mimic joint="index_base_joint" multiplier="1.6" offset="${60 * pi / 180}"/>
+      <mimic joint="index_base_joint" multiplier="1.4" offset="${60 * pi / 180}"/>
     </joint>
     <!-- index base right -->
@@ -126,5 +126,5 @@
       <axis xyz="0 1 0"/>
       <limit effort="1000.0" lower="${0 * pi / 180}" upper="${80 * pi / 180}" velocity="0.8"/>
-      <mimic joint="index_base_joint" multiplier="-1.4" offset="${60 * pi / 180}"/>
+      <mimic joint="index_base_joint" multiplier="-1" offset="${60 * pi / 180}"/>
     </joint>
     <!-- index base right -->

File: hand_robot_ws/src/hand_description/urdf/middle_finger.xacro (robot description, xacro)
@@ -68,5 +68,5 @@
       <axis xyz="0 0 1"/>
       <limit effort="1000.0" lower="${0 * pi / 180}" upper="${130 * pi / 180}" velocity="0.8"/>
-      <mimic joint="middle_base_joint" multiplier="-1.6" offset="${60 * pi / 180}"/>
+      <mimic joint="middle_base_joint" multiplier="-1.4" offset="${60 * pi / 180}"/>
     </joint>
     <!-- middle base right -->
@@ -97,5 +97,5 @@
       <axis xyz="0 0 1"/>
       <limit effort="1000.0" lower="${0 * pi / 180}" upper="${130 * pi / 180}" velocity="0.8"/>
-      <mimic joint="middle_base_joint" multiplier="1.6" offset="${60 * pi / 180}"/>
+      <mimic joint="middle_base_joint" multiplier="1.4" offset="${60 * pi / 180}"/>
     </joint>
     <!-- middle base right -->
@@ -126,5 +126,5 @@
         <axis xyz="0 1 0"/>
         <limit effort="1000.0" lower="${0 * pi / 180}" upper="${80 * pi / 180}" velocity="0.8"/>
-        <mimic joint="middle_base_joint" multiplier="-1.4" offset="${60 * pi / 180}"/>
+        <mimic joint="middle_base_joint" multiplier="-1" offset="${60 * pi / 180}"/>
       </joint>
     <!-- middle base right -->

File: hand_robot_ws/src/hand_description/urdf/pinky_finger.xacro (robot description, xacro)
@@ -62,14 +62,14 @@
       <material>Gazebo/White</material>
     </gazebo>
-    <!-- <joint name="pinky_middle_left_base_left_joint" type="revolute">
-      <origin xyz="-0.052 -0.005 0.006" rpy="${90 * pi / 180} ${70 * pi / 180} 0"/>
+    <joint name="pinky_middle_left_base_left_joint" type="revolute">
+      <origin xyz="-0.033 -0.005 0.003" rpy="${90 * pi / 180} ${70 * pi / 180} 0"/>
       <parent link="pinky_base_left_link"/>
       <child link="pinky_middle_left_link"/>
       <axis xyz="0 0 1"/>
       <limit effort="1000.0" lower="${0 * pi / 180}" upper="${130 * pi / 180}" velocity="0.8"/>
-      <mimic joint="pinky_base_joint" multiplier="-1.6" offset="${60 * pi / 180}"/>
-    </joint> -->
+      <mimic joint="pinky_base_joint" multiplier="-1.4" offset="${60 * pi / 180}"/>
+    </joint>
     <!-- pinky base right -->
-    <!-- <link name="pinky_middle_left_link">
+    <link name="pinky_middle_left_link">
       <visual>
         <geometry>
@@ -77,5 +77,5 @@
         </geometry>
         <material name="white"/>
-        <origin xyz="0.0063 0.0068 -0.0045" rpy="0 0 0"/>
+        <origin xyz="-0.013 0.0 -0.0045" rpy="0 0 0"/>
       </visual>
       <collision>
@@ -86,19 +86,19 @@
       </collision>
       <xacro:cylinder_inertia mass="0.5" radius="0.08" length="0.25"/>
-    </link>  -->
+    </link>
     <!-- Color Gazebo for pinky base right -->
-    <!-- <gazebo reference="pinky_middle_left_link">
+    <gazebo reference="pinky_middle_left_link">
       <material>Gazebo/White</material>
-    </gazebo> -->
-    <!-- <joint name="pinky_middle_right_base_left_joint" type="revolute">
-      <origin xyz="-0.0515 -0.0005 0.012" rpy="${-90 * pi / 180} ${115 * pi / 180} 0"/>
+    </gazebo>
+    <joint name="pinky_middle_right_base_left_joint" type="revolute">
+      <origin xyz="-0.033 -0.0005 0.0088" rpy="${-90 * pi / 180} ${115 * pi / 180} 0"/>
       <parent link="pinky_base_left_link"/>
       <child link="pinky_middle_right_link"/>
       <axis xyz="0 0 1"/>
       <limit effort="1000.0" lower="${0 * pi / 180}" upper="${130 * pi / 180}" velocity="0.8"/>
-      <mimic joint="pinky_base_joint" multiplier="1.6" offset="${60 * pi / 180}"/>
-    </joint> -->
+      <mimic joint="pinky_base_joint" multiplier="1.4" offset="${60 * pi / 180}"/>
+    </joint>
     <!-- pinky base right -->
-    <!-- <link name="pinky_middle_right_link">
+    <link name="pinky_middle_right_link">
       <visual>
         <geometry>
@@ -106,5 +106,5 @@
         </geometry>
         <material name="white"/>
-        <origin xyz="-0.0186 0.0047 0" rpy="0 0 0"/>
+        <origin xyz="0.013 0.00 0" rpy="0 0 0"/>
       </visual>
       <collision>
@@ -115,19 +115,19 @@
       </collision>
       <xacro:cylinder_inertia mass="0.5" radius="0.08" length="0.25"/>
-    </link> -->
+    </link>
     <!-- Color Gazebo for pinky base right -->
-    <!-- <gazebo reference="pinky_middle_left_link">
+    <gazebo reference="pinky_middle_left_link">
       <material>Gazebo/White</material>
-    </gazebo> -->
-    <!-- <joint name="pinky_end_middle_left_joint" type="revolute">
-      <origin xyz="-0.031 0 -0.003" rpy="${90 * pi / 180} ${0 * pi / 180} ${140 * pi / 180}"/>
+    </gazebo>
+    <joint name="pinky_end_middle_left_joint" type="revolute">
+      <origin xyz="-0.025 0 -0.002" rpy="${90 * pi / 180} ${0 * pi / 180} ${140 * pi / 180}"/>
       <parent link="pinky_middle_left_link"/>
       <child link="pinky_end_link"/>
       <axis xyz="0 1 0"/>
       <limit effort="1000.0" lower="${0 * pi / 180}" upper="${80 * pi / 180}" velocity="0.8"/>
-      <mimic joint="pinky_base_joint" multiplier="-1.4" offset="${60 * pi / 180}"/>
-    </joint> -->
+      <mimic joint="pinky_base_joint" multiplier="-1" offset="${60 * pi / 180}"/>
+    </joint>
     <!-- pinky base right -->
-    <!-- <link name="pinky_end_link">
+    <link name="pinky_end_link">
       <visual>
         <geometry>
@@ -135,5 +135,5 @@
         </geometry>
         <material name="white"/>
-        <origin xyz="-0.0241 -0.0156 -0.0058" rpy="0 0 0"/>
+        <origin xyz="0.016 -0.002 -0.0054" rpy="0 0 0"/>
       </visual>
       <collision>
@@ -144,9 +144,9 @@
       </collision>
       <xacro:cylinder_inertia mass="0.5" radius="0.08" length="0.25"/>
-    </link> -->
+    </link>
     <!-- Color Gazebo for pinky base right -->
-    <!-- <gazebo reference="pinky_middle_left_link">
+    <gazebo reference="pinky_middle_left_link">
       <material>Gazebo/White</material>
-    </gazebo> -->
+    </gazebo>
   </xacro:macro>
 </robot>

File: hand_robot_ws/src/hand_description/urdf/ring_finger.xacro (robot description, xacro)
@@ -68,5 +68,5 @@
       <axis xyz="0 0 1"/>
       <limit effort="1000.0" lower="${0 * pi / 180}" upper="${130 * pi / 180}" velocity="0.8"/>
-      <mimic joint="ring_base_joint" multiplier="-1.6" offset="${60 * pi / 180}"/>
+      <mimic joint="ring_base_joint" multiplier="-1.4" offset="${60 * pi / 180}"/>
     </joint>
     <!-- ring base right -->
@@ -97,5 +97,5 @@
       <axis xyz="0 0 1"/>
       <limit effort="1000.0" lower="${0 * pi / 180}" upper="${130 * pi / 180}" velocity="0.8"/>
-      <mimic joint="ring_base_joint" multiplier="1.6" offset="${60 * pi / 180}"/>
+      <mimic joint="ring_base_joint" multiplier="1.4" offset="${60 * pi / 180}"/>
     </joint>
     <!-- ring base right -->
@@ -126,5 +126,5 @@
       <axis xyz="0 1 0"/>
       <limit effort="1000.0" lower="${0 * pi / 180}" upper="${80 * pi / 180}" velocity="0.8"/>
-      <mimic joint="ring_base_joint" multiplier="-1.4" offset="${60 * pi / 180}"/>
+      <mimic joint="ring_base_joint" multiplier="-1" offset="${60 * pi / 180}"/>
     </joint>
     <!-- ring base right -->

File: hand_robot_ws/src/hand_description/urdf/thumb.xacro (robot description, xacro)
@@ -68,5 +68,5 @@
       <axis xyz="0 0 1"/>
       <limit effort="1000.0" lower="${0 * pi / 180}" upper="${130 * pi / 180}" velocity="0.8"/>
-      <mimic joint="thumb_base_joint" multiplier="-1.6" offset="${100 * pi / 180}"/>
+      <mimic joint="thumb_base_joint" multiplier="-1.4" offset="${100 * pi / 180}"/>
     </joint>
     <!-- thumb base right -->
@@ -97,5 +97,5 @@
       <axis xyz="0 0 1"/>
       <limit effort="1000.0" lower="${0 * pi / 180}" upper="${130 * pi / 180}" velocity="0.8"/>
-      <mimic joint="thumb_base_joint" multiplier="1.6" offset="${20 * pi / 180}"/>
+      <mimic joint="thumb_base_joint" multiplier="1.4" offset="${20 * pi / 180}"/>
     </joint>
     <!-- thumb base right -->
@@ -126,5 +126,5 @@
       <axis xyz="0 1 0"/>
       <limit effort="1000.0" lower="${0 * pi / 180}" upper="${80 * pi / 180}" velocity="0.8"/>
-      <mimic joint="thumb_base_joint" multiplier="-1.4" offset="${100 * pi / 180}"/>
+      <mimic joint="thumb_base_joint" multiplier="-1" offset="${140 * pi / 180}"/>
     </joint>
     <!-- thumb base right -->

Commit message: base

File: hand_robot_ws/src/hand_description/urdf/hand.xacro (robot description, xacro)
@@ -14,5 +14,5 @@
   <link name="base_footprint"></link>
   <xacro:forearm parent="base_footprint">
-    <origin xyz="0 0 0" rpy="0 ${90 * pi / 180} 0"/>
+    <origin xyz="-0.044 0 0.13" rpy="0 ${90 * pi / 180} 0"/>
   </xacro:forearm>
   <xacro:wrist parent="horn_link">
