Commit message: palm

File: hand_robot_ws/src/hand_description/urdf/forearm.xacro (robot description, xacro)
@@ -63,5 +63,5 @@
       <origin xyz="0.01 0 0.045" rpy="${180 * pi / 180} 0 0"/>
       <axis xyz="0 0 1"/>
-      <limit effort="10.0" lower="${-180 * pi / 180}" upper="${180 * pi / 180}" velocity="0.3"/>
+      <limit effort="10.0" lower="${-30 * pi / 180}" upper="${90 * pi / 180}" velocity="0.3"/>
     </joint>
     <!-- Servo link -->

File: hand_robot_ws/src/hand_description/urdf/palm.xacro (robot description, xacro)
@@ -36,5 +36,5 @@
       <origin xyz="0 0 0" rpy="0 0 0"/>
       <axis xyz="0 0 1"/>
-      <limit effort="10.0" lower="${-90 * pi / 180}" upper="${90 * pi / 180}" velocity="0.3"/>
+      <limit effort="10.0" lower="${-70 * pi / 180}" upper="${50 * pi / 180}" velocity="0.3"/>
     </joint>
     <!-- Servo link -->

Commit message: base

File: hand_robot_ws/src/hand_description/urdf/forearm.xacro (robot description, xacro)
@@ -16,5 +16,5 @@
         </geometry>
         <material name="white"/>
-        <origin xyz="0 0 0" rpy="0 0 0"/>
+        <origin xyz="-0.044 0 0.13" rpy="0 ${90 * pi / 180} 0"/>
       </visual>
       <collision>
@@ -34,5 +34,5 @@
       <parent link="forearm_link"/>
       <child link="servo_link"/>
-      <origin xyz="-0.0724 -0.039 0.044" rpy="${90 * pi / 180} 0 ${-90 * pi / 180}"/>
+      <origin xyz="0.0 -0.039 0.2" rpy="${0 * pi / 180} 0 ${-90 * pi / 180}"/>
     </joint>
     <!-- Servo link -->

File: hand_robot_ws/src/hand_description/urdf/hand.xacro (robot description, xacro)
@@ -14,5 +14,5 @@
   <link name="base_footprint"></link>
   <xacro:forearm parent="base_footprint">
-    <origin xyz="-0.044 0 0.13" rpy="0 ${90 * pi / 180} 0"/>
+    <origin xyz="0 0 0" rpy="0 ${0 * pi / 180} 0"/>
   </xacro:forearm>
   <xacro:wrist parent="horn_link">

Commit message: base

File: hand_robot_ws/src/hand_description/urdf/forearm.xacro (robot description, xacro)
@@ -4,8 +4,10 @@
   <xacro:macro name="forearm" params="parent *origin">
     <!-- Joint entre base_footprint et forearm -->
-    <joint name="forearm_base_joint_fixed" type="fixed">
+    <joint name="forearm_base_joint" type="revolute">
       <parent link="${parent}"/>
       <child link="forearm_link"/>
       <xacro:insert_block name="origin"/>
+      <axis xyz="0 1 0"/>
+      <limit effort="10.0" lower="${-90 * pi / 180}" upper="${90 * pi / 180}" velocity="0.3"/>
     </joint>
     <!-- Forearm link -->

File: hand_robot_ws/src/hand_description/urdf/hand.xacro (robot description, xacro)
@@ -4,4 +4,5 @@
   <xacro:include filename="$(find hand_description)/urdf/common.xacro"/>
   <xacro:include filename="$(find hand_description)/urdf/ros2_control.xacro"/>
+  <xacro:include filename="$(find hand_description)/urdf/base.xacro"/>
   <xacro:include filename="$(find hand_description)/urdf/forearm.xacro"/>
   <xacro:include filename="$(find hand_description)/urdf/wrist.xacro"/>
@@ -13,6 +14,9 @@
   <xacro:include filename="$(find hand_description)/urdf/pinky_finger.xacro"/>
   <link name="base_footprint"></link>
-  <xacro:forearm parent="base_footprint">
+  <xacro:base parent="base_footprint">
     <origin xyz="0 0 0" rpy="0 ${0 * pi / 180} 0"/>
+  </xacro:base>
+  <xacro:forearm parent="base_rotate_link">
+    <origin xyz="0 0.05 0.03" rpy="0 ${0 * pi / 180} 0"/>
   </xacro:forearm>
   <xacro:wrist parent="horn_link">
